File: electronics/hapy2.5/$brain.sch (KiCad schematic (older format))
At the start: 39 parts, among them P10 WTemp probe, P11 UPPER_BED, P15 Air probe, P19 Power button, P20 T821126A1S100CEU HE10-26, P4 PH Probe, P5 Tank Level Sensor, P6 UPPER_LEDS, P7 LOWER_LEDS, P8 USER_PANEL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

Commit message: post crafty review, wip
Parts:
- gave numbers to parts that had none: 2
Changed lines of the file:
@@
 	4300 2200 4650 2200
 $Comp
-L C C?
+L C C22
 U 1 1 560DEF2B
 P 7450 3150
-F 0 "C?" H 7450 3250 40  0000 L CNN
+F 0 "C22" H 7450 3250 40  0000 L CNN
 F 1 "0.1µF" H 7456 3065 40  0000 L CNN
 F 2 "" H 7488 3000 30  0000 C CNN
@@
 $EndComp
 $Comp
-L C C?
+L C C21
 U 1 1 560DEF5E
 P 7400 5200
-F 0 "C?" H 7400 5300 40  0000 L CNN
+F 0 "C21" H 7400 5300 40  0000 L CNN
 F 1 "0.1µF" H 7406 5115 40  0000 L CNN
 F 2 "" H 7438 5050 30  0000 C CNN
@@
 	7400 5400 7400 5600
 $Comp
-L GND #PWR?
+L GND #PWR23
 U 1 1 560DF36B
 P 7400 5600
-F 0 "#PWR?" H 7400 5600 30  0001 C CNN
+F 0 "#PWR23" H 7400 5600 30  0001 C CNN
 F 1 "GND" H 7400 5530 30  0001 C CNN
 F 2 "" H 7400 5600 60  0000 C CNN
@@
 	7450 3350 7450 3550
 $Comp
-L GND #PWR?
+L GND #PWR24
 U 1 1 560DF7DC
 P 7450 3550
-F 0 "#PWR?" H 7450 3550 30  0001 C CNN
+F 0 "#PWR24" H 7450 3550 30  0001 C CNN
 F 1 "GND" H 7450 3480 30  0001 C CNN
 F 2 "" H 7450 3550 60  0000 C CNN
