File: electronics/hapy2.5/brain.sch (KiCad schematic (older format))
At the start: 39 parts, among them P10 WTemp probe, P11 UPPER_BED, P15 Air probe, P19 Power button, P20 T821126A1S100CEU HE10-26, P4 PH Probe, P5 Tank Level Sensor, P6 UPPER_LEDS, P7 LOWER_LEDS, P8 USER_PANEL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

Commit message: post review schema, cmp and wip pcb
Parts:
- C21, C22: renamed from C?; footprint (none) -> Capacitors_SMD:C_0402
- D17: value ZENER -> MMSZ4678T1G
- R56, R57: footprint (none) -> Resistors_SMD:R_0603
Changed lines of the file:
@@
 5V
 $Comp
-L GND #PWR19
+L GND #PWR019
 U 1 1 55F3CF20
 P 1250 7500
-F 0 "#PWR19" H 1250 7500 30  0001 C CNN
+F 0 "#PWR019" H 1250 7500 30  0001 C CNN
 F 1 "GND" H 1250 7430 30  0001 C CNN
 F 2 "" H 1250 7500 60  0000 C CNN
@@
 P 2150 1650
 F 0 "D17" H 2150 1750 50  0000 C CNN
-F 1 "ZENER" H 2150 1550 40  0000 C CNN
+F 1 "MMSZ4678T1G" H 2150 1550 40  0000 C CNN
 F 2 "risebox:DIODE_SOD-123" H 2150 1650 60  0001 C CNN
 F 3 "" H 2150 1650 60  0000 C CNN
@@
 $EndComp
 $Comp
-L GND #PWR20
+L GND #PWR020
 U 1 1 560BEEB4
 P 2150 2050
-F 0 "#PWR20" H 2150 2050 30  0001 C CNN
+F 0 "#PWR020" H 2150 2050 30  0001 C CNN
 F 1 "GND" H 2150 1980 30  0001 C CNN
 F 2 "" H 2150 2050 60  0000 C CNN
@@
 5V
 $Comp
-L GND #PWR21
+L GND #PWR021
 U 1 1 560C0052
 P 3200 2600
-F 0 "#PWR21" H 3200 2600 30  0001 C CNN
+F 0 "#PWR021" H 3200 2600 30  0001 C CNN
 F 1 "GND" H 3200 2530 30  0001 C CNN
 F 2 "" H 3200 2600 60  0000 C CNN
@@
 F 0 "R56" V 3730 2550 40  0000 C CNN
 F 1 "10K" V 3657 2551 40  0000 C CNN
-F 2 "" V 3580 2550 30  0000 C CNN
+F 2 "Resistors_SMD:R_0603" V 3580 2550 30  0001 C CNN
 F 3 "" H 3650 2550 30  0000 C CNN
 	1    3650 2550
@@
 	3650 2800 3650 2900
 $Comp
-L GND #PWR22
+L GND #PWR022
 U 1 1 560DD230
 P 3650 2900
-F 0 "#PWR22" H 3650 2900 30  0001 C CNN
+F 0 "#PWR022" H 3650 2900 30  0001 C CNN
 F 1 "GND" H 3650 2830 30  0001 C CNN
 F 2 "" H 3650 2900 60  0000 C CNN
@@
 F 0 "R57" V 4130 2200 40  0000 C CNN
 F 1 "100" V 4057 2201 40  0000 C CNN
-F 2 "" V 3980 2200 30  0000 C CNN
+F 2 "Resistors_SMD:R_0603" V 3980 2200 30  0001 C CNN
 F 3 "" H 4050 2200 30  0000 C CNN
 	1    4050 2200
@@
 	4300 2200 4650 2200
 $Comp
-L C C?
+L C C22
 U 1 1 560DEF2B
 P 7450 3150
-F 0 "C?" H 7450 3250 40  0000 L CNN
+F 0 "C22" H 7450 3250 40  0000 L CNN
 F 1 "0.1µF" H 7456 3065 40  0000 L CNN
-F 2 "" H 7488 3000 30  0000 C CNN
+F 2 "Capacitors_SMD:C_0402" H 7488 3000 30  0001 C CNN
 F 3 "" H 7450 3150 60  0000 C CNN
 	1    7450 3150
@@
 $EndComp
 $Comp
-L C C?
+L C C21
 U 1 1 560DEF5E
 P 7400 5200
-F 0 "C?" H 7400 5300 40  0000 L CNN
+F 0 "C21" H 7400 5300 40  0000 L CNN
 F 1 "0.1µF" H 7406 5115 40  0000 L CNN
-F 2 "" H 7438 5050 30  0000 C CNN
+F 2 "Capacitors_SMD:C_0402" H 7438 5050 30  0001 C CNN
 F 3 "" H 7400 5200 60  0000 C CNN
 	1    7400 5200
@@
 	7400 5400 7400 5600
 $Comp
-L GND #PWR?
+L GND #PWR023
 U 1 1 560DF36B
 P 7400 5600
-F 0 "#PWR?" H 7400 5600 30  0001 C CNN
+F 0 "#PWR023" H 7400 5600 30  0001 C CNN
 F 1 "GND" H 7400 5530 30  0001 C CNN
 F 2 "" H 7400 5600 60  0000 C CNN
@@
 	7450 3350 7450 3550
 $Comp
-L GND #PWR?
+L GND #PWR024
 U 1 1 560DF7DC
 P 7450 3550
-F 0 "#PWR?" H 7450 3550 30  0001 C CNN
+F 0 "#PWR024" H 7450 3550 30  0001 C CNN
 F 1 "GND" H 7450 3480 30  0001 C CNN
 F 2 "" H 7450 3550 60  0000 C CNN
