File: electronics/hapy2.5/fans.sch (KiCad schematic (older format))
At the start: 4 parts, among them Q2 2N7002

Commit message: double check all component to footprint matches
Parts:
- D10: footprint Diodes_SMD:SOD-323 -> risebox:DIODE_SOD-323
- Q2: footprint corecode:SOT-23-FET -> risebox:SOT-23-FET
Changed lines of the file:
@@
 F 0 "Q2" H 6510 3870 60  0000 R CNN
 F 1 "2N7002" H 6510 3550 60  0000 R CNN
-F 2 "corecode:SOT-23-FET" H 6500 3700 60  0001 C CNN
+F 2 "risebox:SOT-23-FET" H 6500 3700 60  0001 C CNN
 F 3 "" H 6500 3700 60  0000 C CNN
 	1    6500 3700
@@
 F 0 "D10" H 6950 3150 40  0000 C CNN
 F 1 "PMEG2015EJ,115 DIODE" H 6950 2950 40  0000 C CNN
-F 2 "Diodes_SMD:SOD-323" H 6950 3050 60  0001 C CNN
+F 2 "risebox:DIODE_SOD-323" H 6950 3050 60  0001 C CNN
 F 3 "" H 6950 3050 60  0000 C CNN
 	1    6950 3050

Commit message: post crafty review, wip
Parts:
- Q2: value 2N7002 -> FDN337N
Changed lines of the file:
@@
 $Descr A4 11693 8268
 encoding utf-8
-Sheet 5 7
+Sheet 3 7
 Title ""
 Date ""
@@
 P 6500 3700
 F 0 "Q2" H 6510 3870 60  0000 R CNN
-F 1 "2N7002" H 6510 3550 60  0000 R CNN
+F 1 "FDN337N" H 6510 3550 60  0000 R CNN
 F 2 "risebox:SOT-23-FET" H 6500 3700 60  0001 C CNN
 F 3 "" H 6500 3700 60  0000 C CNN
@@
 	6800 4600 5850 4600
 $Comp
-L GND #PWR014
+L GND #PWR14
 U 1 1 55F27601
 P 5850 4850
-F 0 "#PWR014" H 5850 4850 30  0001 C CNN
+F 0 "#PWR14" H 5850 4850 30  0001 C CNN
 F 1 "GND" H 5850 4780 30  0001 C CNN
 F 2 "" H 5850 4850 60  0000 C CNN
