File: electronics/hapy2.5/main-power.sch (KiCad schematic (older format))
At the start: 21 parts, among them SW1 MSS3112D, U2 DCDC_TI_TPS54335A

Commit message: double check all component to footprint matches
Parts:
- D5: footprint Diodes_SMD:SMB_Standard -> risebox:DIODE_SMB_Standard
Changed lines of the file:
@@
 F 0 "D5" H 3200 3800 50  0000 C CNN
 F 1 "1SMB5935BT3G" H 3200 3600 40  0000 C CNN
-F 2 "Diodes_SMD:SMB_Standard" H 3200 3700 60  0001 C CNN
+F 2 "risebox:DIODE_SMB_Standard" H 3200 3700 60  0001 C CNN
 F 3 "" H 3200 3700 60  0000 C CNN
 	1    3200 3700

Commit message: change C2 footprint to accomodate larger track
Parts:
- C2: footprint Capacitors_SMD:C_0402 -> Capacitors_SMD:C_1206
Changed lines of the file:
@@
 F 0 "C2" H 3600 3800 40  0000 L CNN
 F 1 "10nF" H 3606 3615 40  0000 L CNN
-F 2 "Capacitors_SMD:C_0402" H 3638 3550 30  0001 C CNN
+F 2 "Capacitors_SMD:C_1206" H 3638 3550 30  0001 C CNN
 F 3 "" H 3600 3700 60  0000 C CNN
 	1    3600 3700

Commit message: ajustments
Parts:
- C4: footprint Capacitors_SMD:C_0402 -> Capacitors_SMD:C_1206
- R3: footprint Resistors_SMD:R_0603 -> Resistors_SMD:R_0805
Changed lines of the file:
@@
 F 0 "R3" V 4030 3950 40  0000 C CNN
 F 1 "220K" V 3957 3951 40  0000 C CNN
-F 2 "Resistors_SMD:R_0603" V 3880 3950 30  0001 C CNN
+F 2 "Resistors_SMD:R_0805" V 3880 3950 30  0001 C CNN
 F 3 "" H 3950 3950 30  0000 C CNN
 	1    3950 3950
@@
 F 0 "C4" H 5200 3750 40  0000 L CNN
 F 1 "GMK105BJ104KV-F 0.1µF LE" V 5050 3300 40  0000 L CNN
-F 2 "Capacitors_SMD:C_0402" H 5238 3500 30  0001 C CNN
+F 2 "Capacitors_SMD:C_1206" H 5238 3500 30  0001 C CNN
 F 3 "" H 5200 3650 60  0000 C CNN
 	1    5200 3650

Commit message: post review schema, cmp and wip pcb
Parts:
- D5: value 1SMB5935BT3G -> SMBJ26A Transil; footprint risebox:DIODE_SMB_Standard -> risebox:DIODE_DO_214_AA
Changed lines of the file:
@@
 $EndComp
 $Comp
-L GND #PWR7
+L GND #PWR05
 U 1 1 55F17D04
 P 3950 5800
-F 0 "#PWR7" H 3950 5800 30  0001 C CNN
+F 0 "#PWR05" H 3950 5800 30  0001 C CNN
 F 1 "GND" H 3950 5730 30  0001 C CNN
 F 2 "" H 3950 5800 60  0000 C CNN
@@
 $EndComp
 $Comp
-L GND #PWR8
+L GND #PWR06
 U 1 1 55F17DF2
 P 5200 4250
-F 0 "#PWR8" H 5200 4250 30  0001 C CNN
+F 0 "#PWR06" H 5200 4250 30  0001 C CNN
 F 1 "GND" H 5200 4180 30  0001 C CNN
 F 2 "" H 5200 4250 60  0000 C CNN
@@
 $EndComp
 $Comp
-L GND #PWR9
+L GND #PWR07
 U 1 1 55F17EDD
 P 5850 5800
-F 0 "#PWR9" H 5850 5800 30  0001 C CNN
+F 0 "#PWR07" H 5850 5800 30  0001 C CNN
 F 1 "GND" H 5850 5730 30  0001 C CNN
 F 2 "" H 5850 5800 60  0000 C CNN
@@
 VSENSE
 $Comp
-L GND #PWR10
+L GND #PWR08
 U 1 1 55F17FE2
 P 7850 4100
-F 0 "#PWR10" H 7850 4100 30  0001 C CNN
+F 0 "#PWR08" H 7850 4100 30  0001 C CNN
 F 1 "GND" H 7850 4030 30  0001 C CNN
 F 2 "" H 7850 4100 60  0000 C CNN
@@
 $EndComp
 $Comp
-L GND #PWR11
+L GND #PWR09
 U 1 1 55F18204
 P 8400 5800
-F 0 "#PWR11" H 8400 5800 30  0001 C CNN
+F 0 "#PWR09" H 8400 5800 30  0001 C CNN
 F 1 "GND" H 8400 5730 30  0001 C CNN
 F 2 "" H 8400 5800 60  0000 C CNN
@@
 $EndComp
 $Comp
-L GND #PWR12
+L GND #PWR010
 U 1 1 55F18356
 P 9550 4250
-F 0 "#PWR12" H 9550 4250 30  0001 C CNN
+F 0 "#PWR010" H 9550 4250 30  0001 C CNN
 F 1 "GND" H 9550 4180 30  0001 C CNN
 F 2 "" H 9550 4250 60  0000 C CNN
@@
 $EndComp
 $Comp
-L GND #PWR13
+L GND #PWR011
 U 1 1 55F1A864
 P 10450 6050
-F 0 "#PWR13" H 10450 6050 30  0001 C CNN
+F 0 "#PWR011" H 10450 6050 30  0001 C CNN
 F 1 "GND" H 10450 5980 30  0001 C CNN
 F 2 "" H 10450 6050 60  0000 C CNN
@@
 P 3200 3700
 F 0 "D5" H 3200 3800 50  0000 C CNN
-F 1 "1SMB5935BT3G" H 3200 3600 40  0000 C CNN
-F 2 "risebox:DIODE_SMB_Standard" H 3200 3700 60  0001 C CNN
+F 1 "SMBJ26A  Transil" H 3200 3600 40  0000 C CNN
+F 2 "risebox:DIODE_DO_214_AA" H 3200 3700 60  0001 C CNN
 F 3 "" H 3200 3700 60  0000 C CNN
 	1    3200 3700
@@
 $EndComp
 $Comp
-L GND #PWR6
+L GND #PWR012
 U 1 1 55F22625
 P 2800 4550
-F 0 "#PWR6" H 2800 4550 30  0001 C CNN
+F 0 "#PWR012" H 2800 4550 30  0001 C CNN
 F 1 "GND" H 2800 4480 30  0001 C CNN
 F 2 "" H 2800 4550 60  0000 C CNN
@@
 GNDAlim
 $Comp
-L GND #PWR5
+L GND #PWR013
 U 1 1 55F22765
 P 1450 4550
-F 0 "#PWR5" H 1450 4550 30  0001 C CNN
+F 0 "#PWR013" H 1450 4550 30  0001 C CNN
 F 1 "GND" H 1450 4480 30  0001 C CNN
 F 2 "" H 1450 4550 60  0000 C CNN
