File: electronics/hapy2.5/battery.sch (KiCad schematic (older format))
At the start: 39 parts, among them Q3 BD140, Q4 2N7002, Q5 BSS84P H6327, U3 DCDC_TI_TPS54335A, U5 LM317

Commit message: reduce alim width and add clearance, plus schematics
Parts:
- C10: footprint Capacitors_SMD:C_0402 -> Capacitors_SMD:C_1206
- C13, C14, C15: footprint Capacitors_SMD:C_1206 -> Capacitors_SMD:C_0402
- C18: footprint Capacitors_SMD:C_0402 -> Capacitors_SMD:C_0603
- R10, R11, R39, R44, R47: footprint Resistors_SMD:R_0603 -> Resistors_SMD:R_0805
Changed lines of the file:
@@
 $Descr A4 11693 8268
 encoding utf-8
-Sheet 3 7
+Sheet 7 7
 Title ""
 Date ""
@@
 F 0 "R10" V 5480 5150 40  0000 C CNN
 F 1 "220K" V 5407 5151 40  0000 C CNN
-F 2 "Resistors_SMD:R_0603" V 5330 5150 30  0001 C CNN
+F 2 "Resistors_SMD:R_0805" V 5330 5150 30  0001 C CNN
 F 3 "" H 5400 5150 30  0000 C CNN
 	1    5400 5150
@@
 F 0 "R11" V 5480 5950 40  0000 C CNN
 F 1 "43.2K" V 5407 5951 40  0000 C CNN
-F 2 "Resistors_SMD:R_0603" V 5330 5950 30  0001 C CNN
+F 2 "Resistors_SMD:R_0805" V 5330 5950 30  0001 C CNN
 F 3 "" H 5400 5950 30  0000 C CNN
 	1    5400 5950
@@
 F 0 "C13" H 8000 2900 40  0000 L CNN
 F 1 "GMK105BJ104KV-F 0.1µF LE" H 8006 2715 40  0000 L CNN
-F 2 "Capacitors_SMD:C_1206" H 8038 2650 30  0001 C CNN
+F 2 "Capacitors_SMD:C_0402" H 8038 2650 30  0001 C CNN
 F 3 "" H 8000 2800 60  0000 C CNN
 	1    8000 2800
@@
 F 0 "C14" H 8400 4700 40  0000 L CNN
 F 1 "C0402C120J3GACTU 12pF LE" V 8250 4250 40  0000 L CNN
-F 2 "Capacitors_SMD:C_1206" H 8438 4450 30  0001 C CNN
+F 2 "Capacitors_SMD:C_0402" H 8438 4450 30  0001 C CNN
 F 3 "" H 8400 4600 60  0000 C CNN
 	1    8400 4600
@@
 F 0 "C15" H 9100 4400 40  0000 L CNN
 F 1 "C0402C121J5GACTU 120pF LE" V 9300 3950 40  0000 L CNN
-F 2 "Capacitors_SMD:C_1206" H 9138 4150 30  0001 C CNN
+F 2 "Capacitors_SMD:C_0402" H 9138 4150 30  0001 C CNN
 F 3 "" H 9100 4300 60  0000 C CNN
 	1    9100 4300
@@
 F 0 "C10" H 4000 3500 40  0000 L CNN
 F 1 "10nF" H 4006 3315 40  0000 L CNN
-F 2 "Capacitors_SMD:C_0402" H 4038 3250 30  0001 C CNN
+F 2 "Capacitors_SMD:C_1206" H 4038 3250 30  0001 C CNN
 F 3 "" H 4000 3400 60  0000 C CNN
 	1    4000 3400
@@
 F 0 "R44" V 4130 4700 40  0000 C CNN
 F 1 "10K" V 4057 4701 40  0000 C CNN
-F 2 "Resistors_SMD:R_0603" V 3980 4700 30  0001 C CNN
+F 2 "Resistors_SMD:R_0805" V 3980 4700 30  0001 C CNN
 F 3 "" H 4050 4700 30  0000 C CNN
 	1    4050 4700
@@
 F 0 "R47" V 4780 2150 40  0000 C CNN
 F 1 "11.8K" V 4707 2151 40  0000 C CNN
-F 2 "Resistors_SMD:R_0603" V 4630 2150 30  0001 C CNN
+F 2 "Resistors_SMD:R_0805" V 4630 2150 30  0001 C CNN
 F 3 "" H 4700 2150 30  0000 C CNN
 	1    4700 2150
@@
 F 0 "R39" V 1680 5350 40  0000 C CNN
 F 1 "1K" V 1607 5351 40  0000 C CNN
-F 2 "Resistors_SMD:R_0603" V 1530 5350 30  0001 C CNN
+F 2 "Resistors_SMD:R_0805" V 1530 5350 30  0001 C CNN
 F 3 "" H 1600 5350 30  0000 C CNN
 	1    1600 5350
@@
 F 0 "C18" H 5800 2200 40  0000 L CNN
 F 1 "10nF" H 5806 2015 40  0000 L CNN
-F 2 "Capacitors_SMD:C_0402" H 5838 1950 30  0001 C CNN
+F 2 "Capacitors_SMD:C_0603" H 5838 1950 30  0001 C CNN
 F 3 "" H 5800 2100 60  0000 C CNN
 	1    5800 2100

Commit message: enhanced schema and more room around ph probe slot
Changed lines of the file:
@@
 $EndComp
 $Comp
-L GND #PWR014
+L GND #PWR022
 U 1 1 55F21634
 P 5400 6900
-F 0 "#PWR014" H 5400 6900 30  0001 C CNN
+F 0 "#PWR022" H 5400 6900 30  0001 C CNN
 F 1 "GND" H 5400 6830 30  0001 C CNN
 F 2 "" H 5400 6900 60  0000 C CNN
@@
 $EndComp
 $Comp
-L GND #PWR015
+L GND #PWR023
 U 1 1 55F21649
 P 5400 3950
-F 0 "#PWR015" H 5400 3950 30  0001 C CNN
+F 0 "#PWR023" H 5400 3950 30  0001 C CNN
 F 1 "GND" H 5400 3880 30  0001 C CNN
 F 2 "" H 5400 3950 60  0000 C CNN
@@
 $EndComp
 $Comp
-L GND #PWR016
+L GND #PWR024
 U 1 1 55F21663
 P 6200 4800
-F 0 "#PWR016" H 6200 4800 30  0001 C CNN
+F 0 "#PWR024" H 6200 4800 30  0001 C CNN
 F 1 "GND" H 6200 4730 30  0001 C CNN
 F 2 "" H 6200 4800 60  0000 C CNN
@@
 VSENSE
 $Comp
-L GND #PWR017
+L GND #PWR025
 U 1 1 55F21680
 P 7850 3950
-F 0 "#PWR017" H 7850 3950 30  0001 C CNN
+F 0 "#PWR025" H 7850 3950 30  0001 C CNN
 F 1 "GND" H 7850 3880 30  0001 C CNN
 F 2 "" H 7850 3950 60  0000 C CNN
@@
 $EndComp
 $Comp
-L GND #PWR018
+L GND #PWR026
 U 1 1 55F2169D
 P 8400 5500
-F 0 "#PWR018" H 8400 5500 30  0001 C CNN
+F 0 "#PWR026" H 8400 5500 30  0001 C CNN
 F 1 "GND" H 8400 5430 30  0001 C CNN
 F 2 "" H 8400 5500 60  0000 C CNN
@@
 $EndComp
 $Comp
-L GND #PWR019
+L GND #PWR027
 U 1 1 55F216BF
 P 9550 3950
-F 0 "#PWR019" H 9550 3950 30  0001 C CNN
+F 0 "#PWR027" H 9550 3950 30  0001 C CNN
 F 1 "GND" H 9550 3880 30  0001 C CNN
 F 2 "" H 9550 3950 60  0000 C CNN
@@
 5.4V
 $Comp
-L GND #PWR020
+L GND #PWR028
 U 1 1 55F216FD
 P 10450 5500
-F 0 "#PWR020" H 10450 5500 30  0001 C CNN
+F 0 "#PWR028" H 10450 5500 30  0001 C CNN
 F 1 "GND" H 10450 5430 30  0001 C CNN
 F 2 "" H 10450 5500 60  0000 C CNN
@@
 $EndComp
 $Comp
-L GND #PWR021
+L GND #PWR029
 U 1 1 55F21931
 P 1700 3750
-F 0 "#PWR021" H 1700 3750 30  0001 C CNN
+F 0 "#PWR029" H 1700 3750 30  0001 C CNN
 F 1 "GND" H 1700 3680 30  0001 C CNN
 F 2 "" H 1700 3750 60  0000 C CNN
@@
 $EndComp
 $Comp
-L GND #PWR022
+L GND #PWR030
 U 1 1 55F233C3
 P 3200 4250
-F 0 "#PWR022" H 3200 4250 30  0001 C CNN
+F 0 "#PWR030" H 3200 4250 30  0001 C CNN
 F 1 "GND" H 3200 4180 30  0001 C CNN
 F 2 "" H 3200 4250 60  0000 C CNN
@@
 $EndComp
 $Comp
-L GND #PWR023
+L GND #PWR031
 U 1 1 55F96F04
 P 4600 6900
-F 0 "#PWR023" H 4600 6900 30  0001 C CNN
+F 0 "#PWR031" H 4600 6900 30  0001 C CNN
 F 1 "GND" H 4600 6830 30  0001 C CNN
 F 2 "" H 4600 6900 60  0000 C CNN
@@
 $EndComp
 $Comp
-L GND #PWR024
+L GND #PWR032
 U 1 1 55F9A5CC
 P 4050 1050
-F 0 "#PWR024" H 4050 1050 30  0001 C CNN
+F 0 "#PWR032" H 4050 1050 30  0001 C CNN
 F 1 "GND" H 4050 980 30  0001 C CNN
 F 2 "" H 4050 1050 60  0000 C CNN
@@
 $EndComp
 $Comp
-L GND #PWR025
+L GND #PWR033
 U 1 1 55FAF962
 P 2500 7400
-F 0 "#PWR025" H 2500 7400 30  0001 C CNN
+F 0 "#PWR033" H 2500 7400 30  0001 C CNN
 F 1 "GND" H 2500 7330 30  0001 C CNN
 F 2 "" H 2500 7400 60  0000 C CNN
@@
 $EndComp
 $Comp
-L GND #PWR026
+L GND #PWR034
 U 1 1 55FB0ADB
 P 1050 6750
-F 0 "#PWR026" H 1050 6750 30  0001 C CNN
+F 0 "#PWR034" H 1050 6750 30  0001 C CNN
 F 1 "GND" H 1050 6680 30  0001 C CNN
 F 2 "" H 1050 6750 60  0000 C CNN
@@
 $EndComp
 $Comp
-L GND #PWR027
+L GND #PWR035
 U 1 1 55FB6AB2
 P 3850 7400
-F 0 "#PWR027" H 3850 7400 30  0001 C CNN
+F 0 "#PWR035" H 3850 7400 30  0001 C CNN
 F 1 "GND" H 3850 7330 30  0001 C CNN
 F 2 "" H 3850 7400 60  0000 C CNN
@@
 	5350 2300 5350 2500
 $Comp
-L GND #PWR028
+L GND #PWR036
 U 1 1 55FB7742
 P 5350 2500
-F 0 "#PWR028" H 5350 2500 30  0001 C CNN
+F 0 "#PWR036" H 5350 2500 30  0001 C CNN
 F 1 "GND" H 5350 2430 30  0001 C CNN
 F 2 "" H 5350 2500 60  0000 C CNN
@@
 $EndComp
 $Comp
-L GND #PWR029
+L GND #PWR037
 U 1 1 55FB7756
 P 5800 2500
-F 0 "#PWR029" H 5800 2500 30  0001 C CNN
+F 0 "#PWR037" H 5800 2500 30  0001 C CNN
 F 1 "GND" H 5800 2430 30  0001 C CNN
 F 2 "" H 5800 2500 60  0000 C CNN
@@
 Text Label 2600 2800 0    60   ~ 0
 12V
+Text Notes 800  6200 0    60   ~ 0
+E96
+Text Notes 1350 5400 0    60   ~ 0
+E96
 $EndSCHEMATC

Commit message: fix footprints
Parts:
- C18: footprint Capacitors_SMD:C_0603 -> Capacitors_SMD:C_0402
- R11: footprint Resistors_SMD:R_0805 -> Resistors_SMD:R_0603
- R41: footprint Resistors_SMD:R_0603 -> Resistors_SMD:R_0805
Changed lines of the file:
@@
 F 0 "R11" V 5480 5950 40  0000 C CNN
 F 1 "43.2K" V 5407 5951 40  0000 C CNN
-F 2 "Resistors_SMD:R_0805" V 5330 5950 30  0001 C CNN
+F 2 "Resistors_SMD:R_0603" V 5330 5950 30  0001 C CNN
 F 3 "" H 5400 5950 30  0000 C CNN
 	1    5400 5950
@@
 F 0 "R41" V 2480 5300 40  0000 C CNN
 F 1 "56" V 2407 5301 40  0000 C CNN
-F 2 "Resistors_SMD:R_0603" V 2330 5300 30  0001 C CNN
+F 2 "Resistors_SMD:R_0805" V 2330 5300 30  0001 C CNN
 F 3 "" H 2400 5300 30  0000 C CNN
 	1    2400 5300
@@
 F 0 "C18" H 5800 2200 40  0000 L CNN
 F 1 "10nF" H 5806 2015 40  0000 L CNN
-F 2 "Capacitors_SMD:C_0603" H 5838 1950 30  0001 C CNN
+F 2 "Capacitors_SMD:C_0402" H 5838 1950 30  0001 C CNN
 F 3 "" H 5800 2100 60  0000 C CNN
 	1    5800 2100

Commit message: post crafty review, wip
Parts:
- added C20: 0.1µF, symbol C
- added D18: MRA4007T3G, symbol DIODE
- Q3: value BD140 -> BCP69,115
- R41: footprint Resistors_SMD:R_0805 -> Resistors_SMD:R_1206
Connections:
- net 12V: now also D18.2 (K); no longer Q3.1 (E)
- net Alim24V: now also C20.1
- net GND: now also C20.2
- new net: D18.1 (A), Q3.1 (E)
Other:
- note added: "0.5W"
- note added: "14V, 30mA"
- note removed: "12V, 30mA"
Changed lines of the file:
@@
 $EndComp
 $Comp
-L GND #PWR022
+L GND #PWR32
 U 1 1 55F21634
 P 5400 6900
-F 0 "#PWR022" H 5400 6900 30  0001 C CNN
+F 0 "#PWR32" H 5400 6900 30  0001 C CNN
 F 1 "GND" H 5400 6830 30  0001 C CNN
 F 2 "" H 5400 6900 60  0000 C CNN
@@
 $EndComp
 $Comp
-L GND #PWR023
+L GND #PWR31
 U 1 1 55F21649
 P 5400 3950
-F 0 "#PWR023" H 5400 3950 30  0001 C CNN
+F 0 "#PWR31" H 5400 3950 30  0001 C CNN
 F 1 "GND" H 5400 3880 30  0001 C CNN
 F 2 "" H 5400 3950 60  0000 C CNN
@@
 $EndComp
 $Comp
-L GND #PWR024
+L GND #PWR34
 U 1 1 55F21663
 P 6200 4800
-F 0 "#PWR024" H 6200 4800 30  0001 C CNN
+F 0 "#PWR34" H 6200 4800 30  0001 C CNN
 F 1 "GND" H 6200 4730 30  0001 C CNN
 F 2 "" H 6200 4800 60  0000 C CNN
@@
 VSENSE
 $Comp
-L GND #PWR025
+L GND #PWR35
 U 1 1 55F21680
 P 7850 3950
-F 0 "#PWR025" H 7850 3950 30  0001 C CNN
+F 0 "#PWR35" H 7850 3950 30  0001 C CNN
 F 1 "GND" H 7850 3880 30  0001 C CNN
 F 2 "" H 7850 3950 60  0000 C CNN
@@
 $EndComp
 $Comp
-L GND #PWR026
+L GND #PWR36
 U 1 1 55F2169D
 P 8400 5500
-F 0 "#PWR026" H 8400 5500 30  0001 C CNN
+F 0 "#PWR36" H 8400 5500 30  0001 C CNN
 F 1 "GND" H 8400 5430 30  0001 C CNN
 F 2 "" H 8400 5500 60  0000 C CNN
@@
 $EndComp
 $Comp
-L GND #PWR027
+L GND #PWR37
 U 1 1 55F216BF
 P 9550 3950
-F 0 "#PWR027" H 9550 3950 30  0001 C CNN
+F 0 "#PWR37" H 9550 3950 30  0001 C CNN
 F 1 "GND" H 9550 3880 30  0001 C CNN
 F 2 "" H 9550 3950 60  0000 C CNN
@@
 5.4V
 $Comp
-L GND #PWR028
+L GND #PWR38
 U 1 1 55F216FD
 P 10450 5500
-F 0 "#PWR028" H 10450 5500 30  0001 C CNN
+F 0 "#PWR38" H 10450 5500 30  0001 C CNN
 F 1 "GND" H 10450 5430 30  0001 C CNN
 F 2 "" H 10450 5500 60  0000 C CNN
@@
 $EndComp
 $Comp
-L GND #PWR029
+L GND #PWR24
 U 1 1 55F21931
 P 1700 3750
-F 0 "#PWR029" H 1700 3750 30  0001 C CNN
+F 0 "#PWR24" H 1700 3750 30  0001 C CNN
 F 1 "GND" H 1700 3680 30  0001 C CNN
 F 2 "" H 1700 3750 60  0000 C CNN
@@
 $EndComp
 $Comp
-L GND #PWR030
+L GND #PWR26
 U 1 1 55F233C3
 P 3200 4250
-F 0 "#PWR030" H 3200 4250 30  0001 C CNN
+F 0 "#PWR26" H 3200 4250 30  0001 C CNN
 F 1 "GND" H 3200 4180 30  0001 C CNN
 F 2 "" H 3200 4250 60  0000 C CNN
@@
 $EndComp
 $Comp
-L GND #PWR031
+L GND #PWR29
 U 1 1 55F96F04
 P 4600 6900
-F 0 "#PWR031" H 4600 6900 30  0001 C CNN
+F 0 "#PWR29" H 4600 6900 30  0001 C CNN
 F 1 "GND" H 4600 6830 30  0001 C CNN
 F 2 "" H 4600 6900 60  0000 C CNN
@@
 $EndComp
 $Comp
-L GND #PWR032
+L GND #PWR28
 U 1 1 55F9A5CC
 P 4050 1050
-F 0 "#PWR032" H 4050 1050 30  0001 C CNN
+F 0 "#PWR28" H 4050 1050 30  0001 C CNN
 F 1 "GND" H 4050 980 30  0001 C CNN
 F 2 "" H 4050 1050 60  0000 C CNN
@@
 F 0 "R41" V 2480 5300 40  0000 C CNN
 F 1 "56" V 2407 5301 40  0000 C CNN
-F 2 "Resistors_SMD:R_0805" V 2330 5300 30  0001 C CNN
+F 2 "Resistors_SMD:R_1206" V 2330 5300 30  0001 C CNN
 F 3 "" H 2400 5300 30  0000 C CNN
 	1    2400 5300
@@
 P 2300 6050
 F 0 "Q3" H 2300 5900 40  0000 R CNN
-F 1 "BD140" H 2300 6200 40  0000 R CNN
+F 1 "BCP69,115" H 2300 6200 40  0000 R CNN
 F 2 "Housings_SOT:SOT126_SOT32_Housing_Vertical" H 2180 6150 29  0001 C CNN
 F 3 "" H 2300 6050 60  0000 C CNN
@@
 $EndComp
 $Comp
-L GND #PWR033
+L GND #PWR25
 U 1 1 55FAF962
 P 2500 7400
-F 0 "#PWR033" H 2500 7400 30  0001 C CNN
+F 0 "#PWR25" H 2500 7400 30  0001 C CNN
 F 1 "GND" H 2500 7330 30  0001 C CNN
 F 2 "" H 2500 7400 60  0000 C CNN
@@
 $EndComp
 $Comp
-L GND #PWR034
+L GND #PWR23
 U 1 1 55FB0ADB
 P 1050 6750
-F 0 "#PWR034" H 1050 6750 30  0001 C CNN
+F 0 "#PWR23" H 1050 6750 30  0001 C CNN
 F 1 "GND" H 1050 6680 30  0001 C CNN
 F 2 "" H 1050 6750 60  0000 C CNN
@@
 $EndComp
 Text Notes 2000 4300 0    60   ~ 0
-12V, 30mA
+14V, 30mA
 $Comp
 L R R43
@@
 $EndComp
 $Comp
-L GND #PWR035
+L GND #PWR27
 U 1 1 55FB6AB2
 P 3850 7400
-F 0 "#PWR035" H 3850 7400 30  0001 C CNN
+F 0 "#PWR27" H 3850 7400 30  0001 C CNN
 F 1 "GND" H 3850 7330 30  0001 C CNN
 F 2 "" H 3850 7400 60  0000 C CNN
@@
 Connection ~ 4000 2800
 Wire Wire Line
-	2850 2800 2850 6450
-Connection ~ 2850 2800
-Wire Wire Line
 	2600 2800 6450 2800
 Wire Notes Line
@@
 Connection ~ 4700 1750
 Wire Wire Line
-	2850 6450 2400 6450
+	2400 6450 2900 6450
 Wire Wire Line
 	2400 6450 2400 6250
@@
 Connection ~ 1900 4600
 Wire Wire Line
-	650  4250 650  4600
+	650  4250 650  6600
 Wire Wire Line
 	1050 5100 1050 5900
@@
 	5350 2300 5350 2500
 $Comp
-L GND #PWR036
+L GND #PWR30
 U 1 1 55FB7742
 P 5350 2500
-F 0 "#PWR036" H 5350 2500 30  0001 C CNN
+F 0 "#PWR30" H 5350 2500 30  0001 C CNN
 F 1 "GND" H 5350 2430 30  0001 C CNN
 F 2 "" H 5350 2500 60  0000 C CNN
@@
 $EndComp
 $Comp
-L GND #PWR037
+L GND #PWR33
 U 1 1 55FB7756
 P 5800 2500
-F 0 "#PWR037" H 5800 2500 30  0001 C CNN
+F 0 "#PWR33" H 5800 2500 30  0001 C CNN
 F 1 "GND" H 5800 2430 30  0001 C CNN
 F 2 "" H 5800 2500 60  0000 C CNN
@@
 Text Label 1150 3400 0    60   ~ 0
 GND_battery
-Text Label 2600 2800 0    60   ~ 0
-12V
 Text Notes 800  6200 0    60   ~ 0
 E96
 Text Notes 1350 5400 0    60   ~ 0
 E96
+$Comp
+L DIODE D18
+U 1 1 560D91A1
+P 2900 5800
+F 0 "D18" H 2900 5900 40  0000 C CNN
+F 1 "MRA4007T3G" H 2900 5700 40  0000 C CNN
+F 2 "" H 2900 5800 60  0000 C CNN
+F 3 "" H 2900 5800 60  0000 C CNN
+	1    2900 5800
+	0    -1   -1   0
+$EndComp
+Wire Wire Line
+	650  6600 750  6600
+Connection ~ 650  4600
+$Comp
+L C C20
+U 1 1 560D96CA
+P 750 6800
+F 0 "C20" H 750 6900 40  0000 L CNN
+F 1 "0.1µF" H 756 6715 40  0000 L CNN
+F 2 "" H 788 6650 30  0000 C CNN
+F 3 "" H 750 6800 60  0000 C CNN
+	1    750  6800
+	1    0    0    -1
+$EndComp
+Wire Wire Line
+	750  7000 900  7000
+Wire Wire Line
+	900  7000 900  6600
+Wire Wire Line
+	900  6600 1050 6600
+Connection ~ 1050 6600
+Text Notes 2100 5350 0    60   ~ 0
+0.5W
+Wire Wire Line
+	2900 6450 2900 6000
+Wire Wire Line
+	2900 5600 2900 2800
+Text Label 2600 2800 0    60   ~ 0
+12V
+Connection ~ 2900 2800
 $EndSCHEMATC

Commit message: post review schema, cmp and wip pcb
Parts:
- C20: footprint (none) -> Capacitors_SMD:C_0402
- D18: footprint (none) -> ab2tech:AB2_DO-214AC
- D7: value MMSZ4701-E3-08 ZENER -> SMBJ15A Transil; footprint risebox:DIODE_SOD-123 -> risebox:DIODE_DO_214_AA
- Q3: footprint Housings_SOT:SOT126_SOT32_Housing_Vertical -> ab2tech:AB2_SOT223
- R38: value 9.76K -> 12.4K
- R39: value 1K -> 1.2K
Changed lines of the file:
@@
 $EndComp
 $Comp
-L GND #PWR32
+L GND #PWR025
 U 1 1 55F21634
 P 5400 6900
-F 0 "#PWR32" H 5400 6900 30  0001 C CNN
+F 0 "#PWR025" H 5400 6900 30  0001 C CNN
 F 1 "GND" H 5400 6830 30  0001 C CNN
 F 2 "" H 5400 6900 60  0000 C CNN
@@
 $EndComp
 $Comp
-L GND #PWR31
+L GND #PWR026
 U 1 1 55F21649
 P 5400 3950
-F 0 "#PWR31" H 5400 3950 30  0001 C CNN
+F 0 "#PWR026" H 5400 3950 30  0001 C CNN
 F 1 "GND" H 5400 3880 30  0001 C CNN
 F 2 "" H 5400 3950 60  0000 C CNN
@@
 $EndComp
 $Comp
-L GND #PWR34
+L GND #PWR027
 U 1 1 55F21663
 P 6200 4800
-F 0 "#PWR34" H 6200 4800 30  0001 C CNN
+F 0 "#PWR027" H 6200 4800 30  0001 C CNN
 F 1 "GND" H 6200 4730 30  0001 C CNN
 F 2 "" H 6200 4800 60  0000 C CNN
@@
 VSENSE
 $Comp
-L GND #PWR35
+L GND #PWR028
 U 1 1 55F21680
 P 7850 3950
-F 0 "#PWR35" H 7850 3950 30  0001 C CNN
+F 0 "#PWR028" H 7850 3950 30  0001 C CNN
 F 1 "GND" H 7850 3880 30  0001 C CNN
 F 2 "" H 7850 3950 60  0000 C CNN
@@
 $EndComp
 $Comp
-L GND #PWR36
+L GND #PWR029
 U 1 1 55F2169D
 P 8400 5500
-F 0 "#PWR36" H 8400 5500 30  0001 C CNN
+F 0 "#PWR029" H 8400 5500 30  0001 C CNN
 F 1 "GND" H 8400 5430 30  0001 C CNN
 F 2 "" H 8400 5500 60  0000 C CNN
@@
 $EndComp
 $Comp
-L GND #PWR37
+L GND #PWR030
 U 1 1 55F216BF
 P 9550 3950
-F 0 "#PWR37" H 9550 3950 30  0001 C CNN
+F 0 "#PWR030" H 9550 3950 30  0001 C CNN
 F 1 "GND" H 9550 3880 30  0001 C CNN
 F 2 "" H 9550 3950 60  0000 C CNN
@@
 5.4V
 $Comp
-L GND #PWR38
+L GND #PWR031
 U 1 1 55F216FD
 P 10450 5500
-F 0 "#PWR38" H 10450 5500 30  0001 C CNN
+F 0 "#PWR031" H 10450 5500 30  0001 C CNN
 F 1 "GND" H 10450 5430 30  0001 C CNN
 F 2 "" H 10450 5500 60  0000 C CNN
@@
 $EndComp
 $Comp
-L GND #PWR24
+L GND #PWR032
 U 1 1 55F21931
 P 1700 3750
-F 0 "#PWR24" H 1700 3750 30  0001 C CNN
+F 0 "#PWR032" H 1700 3750 30  0001 C CNN
 F 1 "GND" H 1700 3680 30  0001 C CNN
 F 2 "" H 1700 3750 60  0000 C CNN
@@
 P 3600 3400
 F 0 "D7" H 3600 3500 50  0000 C CNN
-F 1 "MMSZ4701-E3-08 ZENER" H 3600 3300 40  0000 C CNN
-F 2 "risebox:DIODE_SOD-123" H 3600 3400 60  0001 C CNN
+F 1 "SMBJ15A  Transil" H 3600 3300 40  0000 C CNN
+F 2 "risebox:DIODE_DO_214_AA" H 3600 3400 60  0001 C CNN
 F 3 "" H 3600 3400 60  0000 C CNN
 	1    3600 3400
@@
 $EndComp
 $Comp
-L GND #PWR26
+L GND #PWR033
 U 1 1 55F233C3
 P 3200 4250
-F 0 "#PWR26" H 3200 4250 30  0001 C CNN
+F 0 "#PWR033" H 3200 4250 30  0001 C CNN
 F 1 "GND" H 3200 4180 30  0001 C CNN
 F 2 "" H 3200 4250 60  0000 C CNN
@@
 $EndComp
 $Comp
-L GND #PWR29
+L GND #PWR034
 U 1 1 55F96F04
 P 4600 6900
-F 0 "#PWR29" H 4600 6900 30  0001 C CNN
+F 0 "#PWR034" H 4600 6900 30  0001 C CNN
 F 1 "GND" H 4600 6830 30  0001 C CNN
 F 2 "" H 4600 6900 60  0000 C CNN
@@
 $EndComp
 $Comp
-L GND #PWR28
+L GND #PWR035
 U 1 1 55F9A5CC
 P 4050 1050
-F 0 "#PWR28" H 4050 1050 30  0001 C CNN
+F 0 "#PWR035" H 4050 1050 30  0001 C CNN
 F 1 "GND" H 4050 980 30  0001 C CNN
 F 2 "" H 4050 1050 60  0000 C CNN
@@
 F 0 "Q3" H 2300 5900 40  0000 R CNN
 F 1 "BCP69,115" H 2300 6200 40  0000 R CNN
-F 2 "Housings_SOT:SOT126_SOT32_Housing_Vertical" H 2180 6150 29  0001 C CNN
+F 2 "ab2tech:AB2_SOT223" H 2180 6150 29  0001 C CNN
 F 3 "" H 2300 6050 60  0000 C CNN
 	1    2300 6050
@@
 $EndComp
 $Comp
-L GND #PWR25
+L GND #PWR036
 U 1 1 55FAF962
 P 2500 7400
-F 0 "#PWR25" H 2500 7400 30  0001 C CNN
+F 0 "#PWR036" H 2500 7400 30  0001 C CNN
 F 1 "GND" H 2500 7330 30  0001 C CNN
 F 2 "" H 2500 7400 60  0000 C CNN
@@
 P 1600 5350
 F 0 "R39" V 1680 5350 40  0000 C CNN
-F 1 "1K" V 1607 5351 40  0000 C CNN
+F 1 "1.2K" V 1607 5351 40  0000 C CNN
 F 2 "Resistors_SMD:R_0805" V 1530 5350 30  0001 C CNN
 F 3 "" H 1600 5350 30  0000 C CNN
@@
 P 1050 6150
 F 0 "R38" V 1130 6150 40  0000 C CNN
-F 1 "9.76K" V 1057 6151 40  0000 C CNN
+F 1 "12.4K" V 1057 6151 40  0000 C CNN
 F 2 "Resistors_SMD:R_0603" V 980 6150 30  0001 C CNN
 F 3 "" H 1050 6150 30  0000 C CNN
@@
 $EndComp
 $Comp
-L GND #PWR23
+L GND #PWR037
 U 1 1 55FB0ADB
 P 1050 6750
-F 0 "#PWR23" H 1050 6750 30  0001 C CNN
+F 0 "#PWR037" H 1050 6750 30  0001 C CNN
 F 1 "GND" H 1050 6680 30  0001 C CNN
 F 2 "" H 1050 6750 60  0000 C CNN
@@
 $EndComp
 $Comp
-L GND #PWR27
+L GND #PWR038
 U 1 1 55FB6AB2
 P 3850 7400
-F 0 "#PWR27" H 3850 7400 30  0001 C CNN
+F 0 "#PWR038" H 3850 7400 30  0001 C CNN
 F 1 "GND" H 3850 7330 30  0001 C CNN
 F 2 "" H 3850 7400 60  0000 C CNN
@@
 	5350 2300 5350 2500
 $Comp
-L GND #PWR30
+L GND #PWR039
 U 1 1 55FB7742
 P 5350 2500
-F 0 "#PWR30" H 5350 2500 30  0001 C CNN
+F 0 "#PWR039" H 5350 2500 30  0001 C CNN
 F 1 "GND" H 5350 2430 30  0001 C CNN
 F 2 "" H 5350 2500 60  0000 C CNN
@@
 $EndComp
 $Comp
-L GND #PWR33
+L GND #PWR040
 U 1 1 55FB7756
 P 5800 2500
-F 0 "#PWR33" H 5800 2500 30  0001 C CNN
+F 0 "#PWR040" H 5800 2500 30  0001 C CNN
 F 1 "GND" H 5800 2430 30  0001 C CNN
 F 2 "" H 5800 2500 60  0000 C CNN
@@
 F 0 "D18" H 2900 5900 40  0000 C CNN
 F 1 "MRA4007T3G" H 2900 5700 40  0000 C CNN
-F 2 "" H 2900 5800 60  0000 C CNN
+F 2 "ab2tech:AB2_DO-214AC" H 2900 5800 60  0001 C CNN
 F 3 "" H 2900 5800 60  0000 C CNN
 	1    2900 5800
@@
 F 0 "C20" H 750 6900 40  0000 L CNN
 F 1 "0.1µF" H 756 6715 40  0000 L CNN
-F 2 "" H 788 6650 30  0000 C CNN
+F 2 "Capacitors_SMD:C_0402" H 788 6650 30  0001 C CNN
 F 3 "" H 750 6800 60  0000 C CNN
 	1    750  6800

Commit message: fix Q3 PNP and nicer label layouts in progress
Parts:
- C20: footprint Capacitors_SMD:C_0402 -> Capacitors_SMD:C_1206
Changed lines of the file:
@@
 F 0 "C20" H 750 6900 40  0000 L CNN
 F 1 "0.1µF" H 756 6715 40  0000 L CNN
-F 2 "Capacitors_SMD:C_0402" H 788 6650 30  0001 C CNN
+F 2 "Capacitors_SMD:C_1206" H 788 6650 30  0001 C CNN
 F 3 "" H 750 6800 60  0000 C CNN
 	1    750  6800
