File: electronics/indus/leds-controller/Color4.sch (KiCad schematic (older format))
At the start: 0 parts

Commit message: wip review crafty
Other:
- note added: "TODO avec le LM3404 ou avec le TPS92513\nCircuit buck en courant constant 700mA classique (inductance, condos, feedback, boot, PWM, etc)\n"
Changed lines of the file:
@@
 $Descr A4 11693 8268
 encoding utf-8
-Sheet 1 8
-Title ""
+Sheet 6 8
+Title "Carte controlleur de LEDs 4 canaux"
 Date ""
-Rev ""
-Comp ""
+Rev "WIP"
+Comp "Risebox"
 Comment1 ""
 Comment2 ""
@@
 Comment4 ""
 $EndDescr
+Text HLabel 10750 2500 0    60   Output ~ 0
+LED+
+Text HLabel 10750 2750 0    60   Output ~ 0
+LED-
+Text HLabel 1250 2300 0    60   Input ~ 0
+VIN_24V
+Text Notes 3600 3800 0    60   ~ 0
+TODO avec le LM3404 ou avec le TPS92513\nCircuit buck en courant constant 700mA classique (inductance, condos, feedback, boot, PWM, etc)\n
 $EndSCHEMATC

Commit message: wip
Parts:
- added C? (x5): C, symbol C
- added D?: DIODESCH, symbol DIODESCH
- added L?: XAL6060-153MEC - 15µH - 6A, risebox:SELF_COILCRAFT_XAL6060-153, symbol INDUCTOR
- added R? (x6): R, symbol R
- added U?: TPS92513, symbol TPS92513
Connections:
- net LED+: now also C?.1, L?.2
- net LED-: now also C?.2, R?.1, R?.1
- net VIN_24V: now also C?.1, R?.1, R?.2, U?.2 (VIN)
- new net: C?.1, U?.1 (BOOT)
- new net: C?.2, D?.2 (K), L?.1, U?.10 (PH)
- new net: R?.1, R?.2, U?.3 (UVLO)
- new net: R?.1, U?.5 (RT/CLK)
- new net: C?.1, R?.1, U?.6 (IADJ)
- new net: R?.2, U?.7 (ISENSE)
- new net: C?.1, U?.8 (COMP)
- new net GND: C?.2, C?.2, C?.2, D?.1 (A), R?.2, R?.2, R?.2, U?.11 (PAD), U?.9 (GND)
- new net PWM: U?.4 (PDIM)
Other:
- note added: "self métallique"
- note removed: "TODO avec le LM3404 ou avec le TPS92513\nCircuit buck en courant constant 700mA classique (inductance, condos, feedback, boot, PWM, etc)\n"
