File: electronics/indus/leds-controller/fan.sch (KiCad schematic (older format))
At the start: 6 parts

Commit message: more electronic shit
Parts:
- removed D?: KPH-1608EC, risebox:LED_KPH_1608, symbol LED
- removed R?: 470, Resistors_SMD:R_0603, symbol R
Changed lines of the file:
@@
 	6900 3300 6900 3550
 Connection ~ 6900 3550
-$Comp
-L R R?
-U 1 1 57113EAF
-P 4650 4250
-F 0 "R?" V 4730 4250 40  0000 C CNN
-F 1 "470" V 4657 4251 40  0000 C CNN
-F 2 "Resistors_SMD:R_0603" V 4580 4250 30  0001 C CNN
-F 3 "" H 4650 4250 30  0000 C CNN
-	1    4650 4250
-	1    0    0    -1
-$EndComp
-$Comp
-L LED D?
-U 1 1 57113EB0
-P 4650 4900
-F 0 "D?" H 4650 5000 50  0000 C CNN
-F 1 "KPH-1608EC" H 4650 4800 50  0000 C CNN
-F 2 "risebox:LED_KPH_1608" H 4650 4900 60  0001 C CNN
-F 3 "" H 4650 4900 60  0000 C CNN
-	1    4650 4900
-	0    1    1    0
-$EndComp
-$Comp
-L GND #PWR?
-U 1 1 57113EB1
-P 4650 5400
-F 0 "#PWR?" H 4650 5400 30  0001 C CNN
-F 1 "GND" H 4650 5330 30  0001 C CNN
-F 2 "" H 4650 5400 60  0000 C CNN
-F 3 "" H 4650 5400 60  0000 C CNN
-	1    4650 5400
-	1    0    0    -1
-$EndComp
-Wire Wire Line
-	4650 4000 4650 3750
-Connection ~ 4650 3750
-Wire Wire Line
-	4650 4500 4650 4700
-Wire Wire Line
-	4650 5100 4650 5400
 $EndSCHEMATC
