File: electronics/indus/leds-controller/leds-controller.sch (KiCad schematic (older format))
At the start: 16 parts

Commit message: wip review crafty
Parts:
- removed P? (x2): CONN_01X10, symbol CONN_01X10
- added D?: LED, symbol LED
- added P?: ALIM_24V, symbol CONN_01X02
- added P?: CONN_01X02, symbol CONN_01X02
- added P? (x2): CONN_01X11, symbol CONN_01X11
- added R? (x2): R, symbol R
- added TH?: THERMISTOR, symbol THERMISTOR
Connections:
- net ADDR3: now also IC?.9 ((PCINT6/XTAL1/TOSC1)PB6); no longer IC?.19 ((PCINT5/SCK)PB5)
- net ALIM_5V: now also P?.2 (P2), P?.9 (P9)
- net GND: now also D?.2 (K), P?.1 (P1), P?.11 (P11), P?.2 (P2), R?.2
- net TEMP0: now reaches IC?.23 ((PCINT8/ADC0)PC0)
- net TEMP0: now also R?.1, TH?.2
- net TEMP1: now reaches IC?.24 ((PCINT9/ADC1)PC1)
- net TEMP1: now also P?.3 (P3)
- net TEMP2: now reaches IC?.25 ((PCINT10/ADC2)PC2)
- net TEMP2: now also P?.10 (P10)
- new net: IC?.19 ((PCINT5/SCK)PB5), R?.1
- new net: D?.1 (A), R?.2
- new net: P?.10 (P10), P?.2 (P2)
- new net: P?.1 (P1), P?.11 (P11)
- new net: P?.4 (P4), P?.8 (P8)
- new net: P?.3 (P3), P?.9 (P9)
- new net Blue/LED+: P?.5 (P5)
- new net Blue/LED-: P?.6 (P6)
- new net Color3/LED+: P?.6 (P6)
- new net Color3/LED-: P?.7 (P7)
- new net Color4/LED+: P?.7 (P7)
- new net Color4/LED-: P?.8 (P8)
- new net Red/LED+: P?.4 (P4)
- new net Red/LED-: P?.5 (P5)
- new net dcdc_24_12_5/ALIM_24V: P?.1 (P1)
- new net fan/Fan+: P?.1 (P1)
- new net fan/Fan-: P?.2 (P2)
Other:
- note added: "AJOUTER UN QUARTZ\nà 16Meg si besoin"
- moved on the sheet: R?, SW?

Commit message: wip
Connections:
- net ADDR3: now also IC?.13 ((PCINT23/AIN1)PD7); no longer IC?.9 ((PCINT6/XTAL1/TOSC1)PB6)
Other:
- moved on the sheet: D?, R?

Commit message: more electronic shit
Parts:
- removed D? (x2): DIODE, symbol DIODE
- removed P?: CONN_01X02, symbol CONN_01X02
- added C? (x2): 18pF, symbol C
- added P?: CONN_02X03, symbol CONN_02X03
- added SW?: SW_PUSH, symbol SW_PUSH
- added X?: QUARTZCMS4, symbol QUARTZCMS4
- P?: value CONN_01X02 -> CONN_BUS
- P?: symbol CONN_01X11 -> CONN_01X12
- R?: value R -> 10K
- TH?: value THERMISTOR -> THERM CTN 10K
Connections:
- net ADDR1: now also IC?.26 ((PCINT11/ADC3)PC3); no longer IC?.17 ((PCINT3/OC2A/MOSI)PB3)
- net ADDR2: now also IC?.27 ((PCINT12/SDA/ADC4)PC4); no longer IC?.18 ((PCINT4/MISO)PB4)
- net ADDR3: now also IC?.28 ((PCINT14/SCL/ADC5)PC5); no longer IC?.13 ((PCINT23/AIN1)PD7)
- net ALIM_5V: now also IC?.1 ((PCINT14/~RESET~)PC6), R?.1, P?.5 (P5), SW?.1; no longer R?.1, R?.1, R?.1
- net GND: now also IC?.22 (GND), IC?.8 (GND), TH?.2, C?.2, C?.2, SW?.2; no longer R?.2
- net RX: now also U?.1 (RO)
- net TEMP0: now also R?.2, TH?.1; no longer R?.1, TH?.2
- net TX: now also U?.4 (DI)
- net XTAL2: now reaches IC?.10 ((PCINT7/XTAL2/TOSC2)PB7)
- net XTAL2: now also C?.1, X?.1
- net ISC_SCK: now reaches IC?.19 ((PCINT5/SCK)PB5), R?.1
- net ISC_SCK: now also P?.3 (P3)
- net ADDR_5V: now reaches IC?.6 ((PCINT20/XCK/T0)PD4)
- net ADDR_5V: now also R?.1, R?.1, R?.1
- net XTAL1: now reaches IC?.9 ((PCINT6/XTAL1/TOSC1)PB6)
- net XTAL1: now also C?.1, X?.3
- new net ISC_GND: P?.6 (P6)
- new net ISC_MISO: IC?.18 ((PCINT4/MISO)PB4), P?.1 (P1)
- new net ISC_MOSI: IC?.17 ((PCINT3/OC2A/MOSI)PB3), P?.4 (P4)
- new net ISC_VCC: P?.2 (P2)
- no-connect marks 0 -> 4
Other:
- note added: "Ce genre d'alim 5V utilisé \npar moment peut etre mis \nsur une sortie digital\ndu micro"
- note removed: "AJOUTER UN QUARTZ\nà 16Meg si besoin"
- moved on the sheet: P?, R?, TH?
