File: electronics/indus/leds-controller/usb_connector.sch (KiCad schematic (older format))
At the start: 2 parts

Commit message: wip review crafty
Parts:
- added D? (x2): DIODE, symbol DIODE
Connections:
- net at U?.1 (TXD): now also D?.1 (A)
- net VIN_5V: now reaches U?.20 (VCC)
- net at U?.5 (RXD): now also D?.1 (A)
- new net RX: D?.2 (K)
- new net TX: D?.2 (K)
Other:
- note added: "TODO cabler tout ça, en reprennant le schéma de l'arduino nano"
- moved on the sheet: CON?
Changed lines of the file:
@@
 $Descr A4 11693 8268
 encoding utf-8
-Sheet 8 8
-Title ""
+Sheet 7 8
+Title "Carte controlleur de LEDs 4 canaux"
 Date ""
-Rev ""
-Comp ""
+Rev "WIP"
+Comp "Risebox"
 Comment1 ""
 Comment2 ""
@@
 L USB-MINI-B CON?
 U 1 1 570C345D
-P 8700 5100
-F 0 "CON?" H 8450 5550 60  0000 C CNN
-F 1 "USB-MINI-B" H 8650 4600 60  0000 C CNN
-F 2 "" H 8700 5100 60  0000 C CNN
-F 3 "" H 8700 5100 60  0000 C CNN
-	1    8700 5100
+P 2350 4750
+F 0 "CON?" H 2100 5200 60  0000 C CNN
+F 1 "USB-MINI-B" H 2300 4250 60  0000 C CNN
+F 2 "" H 2350 4750 60  0000 C CNN
+F 3 "" H 2350 4750 60  0000 C CNN
+	1    2350 4750
 	1    0    0    -1
 $EndComp
+$Comp
+L DIODE D?
+U 1 1 5711078D
+P 7150 2700
+F 0 "D?" V 7150 2800 40  0000 C CNN
+F 1 "DIODE" H 7150 2600 40  0000 C CNN
+F 2 "" H 7150 2700 60  0000 C CNN
+F 3 "" H 7150 2700 60  0000 C CNN
+	1    7150 2700
+	1    0    0    -1
+$EndComp
+$Comp
+L DIODE D?
+U 1 1 571107E0
+P 7150 3050
+F 0 "D?" H 7150 3150 40  0000 C CNN
+F 1 "DIODE" H 7150 2950 40  0000 C CNN
+F 2 "" H 7150 3050 60  0000 C CNN
+F 3 "" H 7150 3050 60  0000 C CNN
+	1    7150 3050
+	1    0    0    -1
+$EndComp
+Text HLabel 8150 2700 2    60   Output ~ 0
+TX
+Text HLabel 8150 3050 2    60   Input ~ 0
+RX
+Wire Wire Line
+	7350 2700 8150 2700
+Wire Wire Line
+	7350 3050 8150 3050
+Text HLabel 1950 2350 0    60   Input ~ 0
+VIN_5V
+Wire Wire Line
+	1950 2350 3700 2350
+Wire Wire Line
+	3700 2350 3700 2900
+Wire Wire Line
+	3700 2900 4500 2900
+Wire Wire Line
+	6350 2850 6650 2850
+Wire Wire Line
+	6650 2850 6650 2700
+Wire Wire Line
+	6650 2700 6950 2700
+Wire Wire Line
+	6350 2950 6650 2950
+Wire Wire Line
+	6650 2950 6650 3050
+Wire Wire Line
+	6650 3050 6950 3050
+Text Notes 4150 1450 0    60   ~ 0
+TODO cabler tout ça, en reprennant le schéma de l'arduino nano
 $EndSCHEMATC

Commit message: more electronic shit
Parts:
- removed D? (x2): DIODE, symbol DIODE
- added C? (x2): 0.1uF, symbol C
- added C?: 4.7uF, symbol CAPAPOL
- added D? (x2): LED, symbol LED
- added R? (x2): R, symbol R
Connections:
- net RX: now also U?.5 (RXD)
- net TX: now also U?.1 (TXD)
- net VIN_5V: now also U?.4 (VCCIO), D?.1 (A), D?.1 (A)
- net at U?.15 (USBD+): now also CON?.3 (D+)
- net at U?.16 (USBD-): now also CON?.2 (D-)
- net GND: now reaches U?.18 (GND)
- net GND: now also CON?.5 (GND), CON?.6 (SHELL1), CON?.7 (SHELL2), CON?.8 (SHELL3), CON?.9 (SHELL4), U?.21 (GND), U?.25 (AGND), U?.7 (GND), C?.2, C?.2
- net at U?.2 (DTR): now also C?.2
- net at U?.22 (CBUS1): now also R?.2
- net at U?.23 (CBUS0): now also R?.2
- net VUSB: now reaches CON?.1 (VBUS)
- net VUSB: now also C?.1, C?.1
- new net: D?.2 (K), R?.1 (x2)
- new net RESET_MCU: C?.1
- no-connect marks 0 -> 14
Other:
- note added: "Attention à l'alim par usb : est-ce que je la drope ou pas. Autre idée : court circuiter 2 pattes pour le passer en mode test."
- moved on the sheet: CON?
