File: electronics/indus/leds/leds.sch (KiCad schematic (older format))
At the start: 18 parts

Commit message: wip
Parts:
- removed P?: CONN_01X10, symbol CONN_01X10
- added P?: CONN_01X11, symbol CONN_01X11
Connections:
- net at D?.1 (A): now also P?.11 (P11)
- net at D?.2 (K): now also P?.4 (P4)
- net at D?.2 (K): now also P?.5 (P5)
- net at D?.2 (K): now also P?.6 (P6)
- net at D?.2 (K): now also P?.7 (P7)
- net at TH?.1: now also P?.2 (P2)
- net at TH?.2: now also P?.3 (P3)
- net at D?.1 (A): now also P?.8 (P8)
- net at D?.1 (A): now also P?.9 (P9)
- net at D?.1 (A): now also P?.10 (P10)
- new net GND: P?.1 (P1)
Other:
- moved on the sheet: D?, TH?

Commit message: more electronic shit
Parts:
- added R?: 10K, symbol R
- P1: renamed from P?; symbol CONN_01X11 -> CONN_01X12
- TH1: renamed from TH?; value THERMISTOR -> THERM CTN 10K
- gave numbers to parts that had none: 16
Connections:
- net GND: now also P1.2 (P2), TH1.1; no longer P1.1 (P1)
- net at D1.1 (A): now also P1.12 (P12); no longer P1.11 (P11)
- net at D13.2 (K): now also P1.5 (P5); no longer P1.4 (P4)
- net at D2.1 (A): now also P1.11 (P11); no longer P1.10 (P10)
- net at D14.2 (K): now also P1.6 (P6); no longer P1.5 (P5)
- net at D3.1 (A): now also P1.10 (P10); no longer P1.9 (P9)
- net at D15.2 (K): now also P1.7 (P7); no longer P1.6 (P6)
- net at D4.1 (A): now also P1.9 (P9); no longer P1.8 (P8)
- net at D16.2 (K): now also P1.8 (P8); no longer P1.7 (P7)
- net at P1.3 (P3), TH1.2: now also R?.2
- new net: P1.4 (P4), R?.1
- no-connect marks 0 -> 1
Other:
- moved on the sheet: TH1
Changed lines of the file:
@@
 $EndDescr
 $Comp
-L LED D?
+L LED D1
 U 1 1 56E1A1EF
 P 3050 2250
-F 0 "D?" H 3050 2350 50  0000 C CNN
+F 0 "D1" H 3050 2350 50  0000 C CNN
 F 1 "LED" H 3050 2150 50  0000 C CNN
 F 2 "" H 3050 2250 60  0000 C CNN
@@
 $EndComp
 $Comp
-L LED D?
+L LED D5
 U 1 1 56E1A231
 P 3700 2250
-F 0 "D?" H 3700 2350 50  0000 C CNN
+F 0 "D5" H 3700 2350 50  0000 C CNN
 F 1 "LED" H 3700 2150 50  0000 C CNN
 F 2 "" H 3700 2250 60  0000 C CNN
@@
 $EndComp
 $Comp
-L LED D?
+L LED D9
 U 1 1 56E1A294
 P 4350 2250
-F 0 "D?" H 4350 2350 50  0000 C CNN
+F 0 "D9" H 4350 2350 50  0000 C CNN
 F 1 "LED" H 4350 2150 50  0000 C CNN
 F 2 "" H 4350 2250 60  0000 C CNN
@@
 $EndComp
 $Comp
-L LED D?
+L LED D13
 U 1 1 56E1A2C5
 P 5000 2250
-F 0 "D?" H 5000 2350 50  0000 C CNN
+F 0 "D13" H 5000 2350 50  0000 C CNN
 F 1 "LED" H 5000 2150 50  0000 C CNN
 F 2 "" H 5000 2250 60  0000 C CNN
@@
 $EndComp
 $Comp
-L LED D?
+L LED D2
 U 1 1 56E1BEDB
 P 3050 2750
-F 0 "D?" H 3050 2850 50  0000 C CNN
+F 0 "D2" H 3050 2850 50  0000 C CNN
 F 1 "LED" H 3050 2650 50  0000 C CNN
 F 2 "" H 3050 2750 60  0000 C CNN
@@
 $EndComp
 $Comp
-L LED D?
+L LED D6
 U 1 1 56E1BEE1
 P 3700 2750
-F 0 "D?" H 3700 2850 50  0000 C CNN
+F 0 "D6" H 3700 2850 50  0000 C CNN
 F 1 "LED" H 3700 2650 50  0000 C CNN
 F 2 "" H 3700 2750 60  0000 C CNN
@@
 $EndComp
 $Comp
-L LED D?
+L LED D10
 U 1 1 56E1BEE7
 P 4350 2750
-F 0 "D?" H 4350 2850 50  0000 C CNN
+F 0 "D10" H 4350 2850 50  0000 C CNN
 F 1 "LED" H 4350 2650 50  0000 C CNN
 F 2 "" H 4350 2750 60  0000 C CNN
@@
 $EndComp
 $Comp
-L LED D?
+L LED D14
 U 1 1 56E1BEED
 P 5000 2750
-F 0 "D?" H 5000 2850 50  0000 C CNN
+F 0 "D14" H 5000 2850 50  0000 C CNN
 F 1 "LED" H 5000 2650 50  0000 C CNN
 F 2 "" H 5000 2750 60  0000 C CNN
@@
 $EndComp
 $Comp
-L LED D?
+L LED D3
 U 1 1 56E1C418
 P 3050 3250
-F 0 "D?" H 3050 3350 50  0000 C CNN
+F 0 "D3" H 3050 3350 50  0000 C CNN
 F 1 "LED" H 3050 3150 50  0000 C CNN
 F 2 "" H 3050 3250 60  0000 C CNN
@@
 $EndComp
 $Comp
-L LED D?
+L LED D7
 U 1 1 56E1C41E
 P 3700 3250
-F 0 "D?" H 3700 3350 50  0000 C CNN
+F 0 "D7" H 3700 3350 50  0000 C CNN
 F 1 "LED" H 3700 3150 50  0000 C CNN
 F 2 "" H 3700 3250 60  0000 C CNN
@@
 $EndComp
 $Comp
-L LED D?
+L LED D11
 U 1 1 56E1C424
 P 4350 3250
-F 0 "D?" H 4350 3350 50  0000 C CNN
+F 0 "D11" H 4350 3350 50  0000 C CNN
 F 1 "LED" H 4350 3150 50  0000 C CNN
 F 2 "" H 4350 3250 60  0000 C CNN
@@
 $EndComp
 $Comp
-L LED D?
+L LED D15
 U 1 1 56E1C42A
 P 5000 3250
-F 0 "D?" H 5000 3350 50  0000 C CNN
+F 0 "D15" H 5000 3350 50  0000 C CNN
 F 1 "LED" H 5000 3150 50  0000 C CNN
 F 2 "" H 5000 3250 60  0000 C CNN
@@
 $EndComp
 $Comp
-L LED D?
+L LED D4
 U 1 1 56E1C44F
 P 3050 3750
-F 0 "D?" H 3050 3850 50  0000 C CNN
+F 0 "D4" H 3050 3850 50  0000 C CNN
 F 1 "LED" H 3050 3650 50  0000 C CNN
 F 2 "" H 3050 3750 60  0000 C CNN
@@
 $EndComp
 $Comp
-L LED D?
+L LED D8
 U 1 1 56E1C455
 P 3700 3750
-F 0 "D?" H 3700 3850 50  0000 C CNN
+F 0 "D8" H 3700 3850 50  0000 C CNN
 F 1 "LED" H 3700 3650 50  0000 C CNN
 F 2 "" H 3700 3750 60  0000 C CNN
@@
 $EndComp
 $Comp
-L LED D?
+L LED D12
 U 1 1 56E1C45B
 P 4350 3750
-F 0 "D?" H 4350 3850 50  0000 C CNN
+F 0 "D12" H 4350 3850 50  0000 C CNN
 F 1 "LED" H 4350 3650 50  0000 C CNN
 F 2 "" H 4350 3750 60  0000 C CNN
@@
 $EndComp
 $Comp
-L LED D?
+L LED D16
 U 1 1 56E1C461
 P 5000 3750
-F 0 "D?" H 5000 3850 50  0000 C CNN
+F 0 "D16" H 5000 3850 50  0000 C CNN
 F 1 "LED" H 5000 3650 50  0000 C CNN
 F 2 "" H 5000 3750 60  0000 C CNN
@@
 $EndComp
 $Comp
-L THERMISTOR TH?
+L THERMISTOR TH1
 U 1 1 56E1CF63
-P 6300 4800
-F 0 "TH?" V 6400 4850 50  0000 C CNN
-F 1 "THERMISTOR" V 6200 4800 50  0000 C CNN
-F 2 "" H 6300 4800 60  0000 C CNN
-F 3 "" H 6300 4800 60  0000 C CNN
-	1    6300 4800
+P 7000 4800
+F 0 "TH1" V 7100 4850 50  0000 C CNN
+F 1 "THERM CTN 10K" V 6900 4800 50  0000 C CNN
+F 2 "" H 7000 4800 60  0000 C CNN
+F 3 "" H 7000 4800 60  0000 C CNN
+	1    7000 4800
 	0    1    1    0
 $EndComp
@@
 	5950 3750 5200 3750
 $Comp
-L CONN_01X11 P?
+L CONN_01X12 P1
 U 1 1 5714EB1D
-P 5050 5400
-F 0 "P?" H 5050 6000 50  0000 C CNN
-F 1 "CONN_01X11" V 5150 5400 50  0000 C CNN
-F 2 "" H 5050 5400 60  0000 C CNN
-F 3 "" H 5050 5400 60  0000 C CNN
-	1    5050 5400
+P 5100 5400
+F 0 "P1" H 5100 6000 50  0000 C CNN
+F 1 "CONN_01X11" V 5200 5400 50  0000 C CNN
+F 2 "" H 5100 5400 60  0000 C CNN
+F 3 "" H 5100 5400 60  0000 C CNN
+	1    5100 5400
 	0    1    1    0
 $EndComp
@@
 	5350 4800 5350 5200
 Wire Wire Line
-	5350 4800 6050 4800
-Wire Wire Line
-	6550 4800 6900 4800
-Wire Wire Line
-	6900 4800 6900 5000
-Wire Wire Line
-	6900 5000 5450 5000
-Wire Wire Line
-	5450 5000 5450 5200
-$Comp
-L GND #PWR?
+	5450 4950 5450 5200
+$Comp
+L GND #PWR1
 U 1 1 5714EE15
-P 6300 5600
-F 0 "#PWR?" H 6300 5600 30  0001 C CNN
-F 1 "GND" H 6300 5530 30  0001 C CNN
-F 2 "" H 6300 5600 60  0000 C CNN
-F 3 "" H 6300 5600 60  0000 C CNN
-	1    6300 5600
+P 6500 5600
+F 0 "#PWR1" H 6500 5600 30  0001 C CNN
+F 1 "GND" H 6500 5530 30  0001 C CNN
+F 2 "" H 6500 5600 60  0000 C CNN
+F 3 "" H 6500 5600 60  0000 C CNN
+	1    6500 5600
 	1    0    0    -1
 $EndComp
@@
 	5550 5200 5550 5100
 Wire Wire Line
-	5550 5100 6300 5100
-Wire Wire Line
-	6300 5100 6300 5600
+	5550 5100 7550 5100
+$Comp
+L R R?
+U 1 1 574515E8
+P 6000 4800
+F 0 "R?" V 6080 4800 40  0000 C CNN
+F 1 "10K" V 6007 4801 40  0000 C CNN
+F 2 "" V 5930 4800 30  0000 C CNN
+F 3 "" H 6000 4800 30  0000 C CNN
+	1    6000 4800
+	0    -1   -1   0
+$EndComp
+Wire Wire Line
+	7250 4800 7550 4800
+Wire Wire Line
+	7550 4800 7550 5100
+Wire Wire Line
+	5350 4800 5750 4800
+Wire Wire Line
+	6250 4800 6750 4800
+Wire Wire Line
+	5450 4950 6500 4950
+Wire Wire Line
+	6500 4950 6500 4800
+Connection ~ 6500 4800
+Wire Wire Line
+	6500 5600 6500 5100
+Connection ~ 6500 5100
+NoConn ~ 5650 5200
 $EndSCHEMATC
