File: electronics/indus/leds-controller_diy/leds-controller.sch (KiCad schematic (older format))
At the start: 24 parts

Commit message: wip bare diy controller
Parts:
- C? (x3): symbol C -> C-RESCUE-leds-controller
- D?: symbol LED -> LED-RESCUE-leds-controller
- IC?: symbol ATMEGA328-P -> ATMEGA328-P-RESCUE-leds-controller
- R? (x7): symbol R -> R-RESCUE-leds-controller
Changed lines of the file:
@@
 EESchema Schematic File Version 2
+LIBS:leds-controller-rescue
 LIBS:power
 LIBS:device
@@
 LIBS:memory
 LIBS:xilinx
-LIBS:special
 LIBS:microcontrollers
 LIBS:dsp
@@
 $EndDescr
 $Comp
-L ATMEGA328-P IC?
+L ATMEGA328-P-RESCUE-leds-controller IC?
 U 1 1 56E1DAFD
 P 3950 3750
@@
 $EndComp
 $Comp
-L GND #PWR?
+L GND-RESCUE-leds-controller #PWR?
 U 1 1 56E1DB95
 P 700 800
@@
 $EndComp
 $Comp
-L GND #PWR?
+L GND-RESCUE-leds-controller #PWR?
 U 1 1 56E1F01C
 P 1250 5050
@@
 $EndComp
 $Comp
-L R R?
+L R-RESCUE-leds-controller R?
 U 1 1 56E1F0BA
 P 1000 3800
@@
 $EndComp
 $Comp
-L R R?
+L R-RESCUE-leds-controller R?
 U 1 1 56E1F0F6
 P 1250 3800
@@
 $EndComp
 $Comp
-L R R?
+L R-RESCUE-leds-controller R?
 U 1 1 56E1F119
 P 1500 3800
@@
 TX
 $Comp
-L R R?
+L R-RESCUE-leds-controller R?
 U 1 1 570C2C8C
 P 1950 2650
@@
 $EndComp
 $Comp
-L C C?
+L C-RESCUE-leds-controller C?
 U 1 1 570C2CB7
 P 1400 2300
@@
 $EndComp
 $Comp
-L GND #PWR?
+L GND-RESCUE-leds-controller #PWR?
 U 1 1 570C3013
 P 850 2150
@@
 $EndSheet
 $Comp
-L R R?
+L R-RESCUE-leds-controller R?
 U 1 1 570C3845
 P 4600 5800
@@
 ALIM_5V
 $Comp
-L GND #PWR?
+L GND-RESCUE-leds-controller #PWR?
 U 1 1 570FC0EA
 P 2100 1300
@@
 ALIM_12V
 $Comp
-L LED D?
+L LED-RESCUE-leds-controller D?
 U 1 1 5710F8AD
 P 6100 2550
@@
 $EndComp
 $Comp
-L GND #PWR?
+L GND-RESCUE-leds-controller #PWR?
 U 1 1 5710F8D8
 P 6300 2700
@@
 $EndComp
 $Comp
-L R R?
+L R-RESCUE-leds-controller R?
 U 1 1 5710F961
 P 5900 2900
@@
 TEMP2
 $Comp
-L GND #PWR?
+L GND-RESCUE-leds-controller #PWR?
 U 1 1 57118968
 P 10100 6000
@@
 $EndComp
 $Comp
-L GND #PWR?
+L GND-RESCUE-leds-controller #PWR?
 U 1 1 5714DE0B
 P 9500 2500
@@
 $EndComp
 $Comp
-L R R?
+L R-RESCUE-leds-controller R?
 U 1 1 5714EAA9
 P 5650 1100
@@
 $EndComp
 $Comp
-L GND #PWR?
+L GND-RESCUE-leds-controller #PWR?
 U 1 1 5714EACC
 P 5650 2350
@@
 $EndComp
 $Comp
-L C C?
+L C-RESCUE-leds-controller C?
 U 1 1 572988EA
 P 2800 5450
@@
 $EndComp
 $Comp
-L C C?
+L C-RESCUE-leds-controller C?
 U 1 1 57298990
 P 1800 5450
@@
 	2800 5800 2800 5650
 $Comp
-L GND #PWR?
+L GND-RESCUE-leds-controller #PWR?
 U 1 1 5729D841
 P 2300 6000
@@
 NoConn ~ 3050 3250
 $Comp
-L GND #PWR?
+L GND-RESCUE-leds-controller #PWR?
 U 1 1 57448CD8
 P 2950 5150
@@
 	6700 4100 6700 4300
 $Comp
-L GND #PWR?
+L GND-RESCUE-leds-controller #PWR?
 U 1 1 5744AD3B
 P 6700 4300
