File: electronics/indus/leds-controller_diy_bare/dcdc_24_5.sch (KiCad schematic (older format))
At the start: 20 parts

Commit message: wip bare diy controller
Parts:
- removed U?: 7805, symbol 7805
- C? (x8): symbol C-RESCUE-leds-controller -> C
- D?: symbol ZENER-RESCUE-leds-controller -> ZENER
- R? (x7): symbol R-RESCUE-leds-controller -> R
Connections:
- net labels added: ALIM_24V+
- net labels removed: 5V, ALIM_24V
- wire segments 53 -> 69
Changed lines of the file:
@@
 EESchema Schematic File Version 2
-LIBS:leds-controller-rescue
 LIBS:power
 LIBS:device
@@
 LIBS:memory
 LIBS:xilinx
+LIBS:special
 LIBS:microcontrollers
 LIBS:dsp
@@
 encoding utf-8
 Sheet 2 8
-Title "Carte controlleur de LEDs 4 canaux"
+Title ""
 Date ""
-Rev "WIP"
-Comp "Risebox"
+Rev ""
+Comp ""
 Comment1 ""
 Comment2 ""
@@
 $EndDescr
 $Comp
-L R-RESCUE-leds-controller R?
+L R R?
 U 1 1 570BE927
 P 3250 3800
@@
 $EndComp
 $Comp
-L R-RESCUE-leds-controller R?
+L R R?
 U 1 1 570BE928
 P 3250 4600
@@
 $EndComp
 $Comp
-L GND-RESCUE-leds-controller #PWR?
+L GND #PWR?
 U 1 1 570BE929
 P 3250 5350
@@
 $EndComp
 $Comp
-L C-RESCUE-leds-controller C?
+L C C?
 U 1 1 570BE92A
 P 3850 3050
@@
 $EndComp
 $Comp
-L C-RESCUE-leds-controller C?
+L C C?
 U 1 1 570BE92B
 P 4250 3050
@@
 $EndComp
 $Comp
-L GND-RESCUE-leds-controller #PWR?
+L GND #PWR?
 U 1 1 570BE92C
 P 4250 3650
@@
 $EndComp
 $Comp
-L R-RESCUE-leds-controller R?
+L R R?
 U 1 1 570BE92D
 P 5050 3850
@@
 $EndComp
 $Comp
-L GND-RESCUE-leds-controller #PWR?
+L GND #PWR?
 U 1 1 570BE92E
 P 5050 4500
@@
 $EndComp
 $Comp
-L C-RESCUE-leds-controller C?
+L C C?
 U 1 1 570BE92F
 P 6850 2500
@@
 VSENSE
 $Comp
-L GND-RESCUE-leds-controller #PWR?
+L GND #PWR?
 U 1 1 570BE931
 P 6700 3650
@@
 $EndComp
 $Comp
-L R-RESCUE-leds-controller R?
+L R R?
 U 1 1 570BE932
 P 7250 3550
@@
 $EndComp
 $Comp
-L C-RESCUE-leds-controller C?
+L C C?
 U 1 1 570BE933
 P 7250 4300
@@
 $EndComp
 $Comp
-L GND-RESCUE-leds-controller #PWR?
+L GND #PWR?
 U 1 1 570BE934
 P 7250 5200
@@
 $EndComp
 $Comp
-L C-RESCUE-leds-controller C?
+L C C?
 U 1 1 570BE935
 P 7950 4000
@@
 $EndComp
 $Comp
-L C-RESCUE-leds-controller C?
+L C C?
 U 1 1 570BE936
 P 8400 3000
@@
 $EndComp
 $Comp
-L C-RESCUE-leds-controller C?
+L C C?
 U 1 1 570BE937
 P 8850 3000
@@
 $EndComp
 $Comp
-L GND-RESCUE-leds-controller #PWR?
+L GND #PWR?
 U 1 1 570BE938
 P 8400 3650
@@
 $EndComp
 $Comp
-L R-RESCUE-leds-controller R?
+L R R?
 U 1 1 570BE939
 P 9300 3000
@@
 $EndComp
 $Comp
-L R-RESCUE-leds-controller R?
+L R R?
 U 1 1 570BE93A
 P 9300 3750
@@
 $EndComp
 $Comp
-L R-RESCUE-leds-controller R?
+L R R?
 U 1 1 570BE93B
 P 9300 4650
@@
 Text Label 9450 4200 0    60   ~ 0
 VSENSE
-Text HLabel 10850 2500 2    60   Output ~ 0
+Text HLabel 10050 2500 2    60   Output ~ 0
 12V
 $Comp
-L GND-RESCUE-leds-controller #PWR?
+L GND #PWR?
 U 1 1 570BE93C
 P 9300 5200
@@
 $EndComp
 $Comp
-L ZENER-RESCUE-leds-controller D?
+L ZENER D?
 U 1 1 570BE941
 P 2450 3100
@@
 $EndComp
 $Comp
-L C-RESCUE-leds-controller C?
+L C C?
 U 1 1 570BE942
 P 2850 3100
@@
 $EndComp
 $Comp
-L GND-RESCUE-leds-controller #PWR?
+L GND #PWR?
 U 1 1 570BE943
 P 2050 3950
@@
 $EndComp
 Text HLabel 1550 2500 0    60   Input ~ 0
-ALIM_24V
-Wire Wire Line
-	3250 4050 3250 4350
+ALIM_24V+
+Wire Wire Line
+	3250 4050 3250 4200
+Wire Wire Line
+	3250 4200 3250 4350
 Wire Wire Line
 	3250 4850 3250 5350
@@
 	3850 3400 4250 3400
 Wire Wire Line
-	4250 3250 4250 3650
+	4250 3250 4250 3400
+Wire Wire Line
+	4250 3400 4250 3650
 Wire Wire Line
 	4250 2500 4250 2850
@@
 	6300 2500 6650 2500
 Wire Wire Line
-	7050 2500 7450 2500
+	7050 2500 7250 2500
+Wire Wire Line
+	7250 2500 7450 2500
 Wire Wire Line
 	6300 2700 7250 2700
@@
 	6300 3100 6700 3100
 Wire Wire Line
-	6700 3100 6700 3650
+	6700 3100 6700 3200
+Wire Wire Line
+	6700 3200 6700 3650
 Wire Wire Line
 	6300 3200 6700 3200
 Connection ~ 6700 3200
 Wire Wire Line
-	6300 2900 7950 2900
+	6300 2900 7250 2900
+Wire Wire Line
+	7250 2900 7950 2900
 Wire Wire Line
 	7250 2900 7250 3300
@@
 	7250 3800 7250 4100
 Wire Wire Line
-	7250 4500 7250 5200
+	7250 4500 7250 4700
+Wire Wire Line
+	7250 4700 7250 5200
 Wire Wire Line
 	7950 2900 7950 3800
@@
 Connection ~ 7250 4700
 Wire Wire Line
-	8050 2500 10850 2500
+	8050 2500 8400 2500
+Wire Wire Line
+	8400 2500 8850 2500
+Wire Wire Line
+	8850 2500 9300 2500
+Wire Wire Line
+	9300 2500 10050 2500
 Wire Wire Line
 	8400 2800 8400 2500
@@
 Connection ~ 8850 2500
 Wire Wire Line
-	8400 3200 8400 3650
+	8400 3200 8400 3450
+Wire Wire Line
+	8400 3450 8400 3650
 Wire Wire Line
 	8850 3200 8850 3450
@@
 	9300 3250 9300 3500
 Wire Wire Line
-	9300 4000 9300 4400
+	9300 4000 9300 4200
+Wire Wire Line
+	9300 4200 9300 4400
 Wire Wire Line
 	9300 4200 9800 4200
@@
 	2850 2500 2850 2900
 Wire Wire Line
-	2050 3300 2050 3950
+	2050 3300 2050 3600
+Wire Wire Line
+	2050 3600 2050 3950
 Wire Wire Line
 	2450 3600 2450 3300
 Wire Wire Line
-	2000 3600 2850 3600
+	2000 3600 2050 3600
+Wire Wire Line
+	2050 3600 2450 3600
+Wire Wire Line
+	2450 3600 2850 3600
 Connection ~ 2050 3600
 Wire Wire Line
@@
 	8200 2700 8200 2550
 Wire Wire Line
-	1550 2500 5300 2500
+	1550 2500 2050 2500
+Wire Wire Line
+	2050 2500 2450 2500
+Wire Wire Line
+	2450 2500 2850 2500
+Wire Wire Line
+	2850 2500 3250 2500
+Wire Wire Line
+	3250 2500 3550 2500
+Wire Wire Line
+	3550 2500 3850 2500
+Wire Wire Line
+	3850 2500 4250 2500
+Wire Wire Line
+	4250 2500 5300 2500
 Wire Wire Line
 	4750 2900 4750 4200
@@
 Text Notes 7550 5500 0    60   ~ 0
 TODO : Ajuster pour sortir à 12V
-$Comp
-L 7805 U?
-U 1 1 570FB25B
-P 10350 3350
-F 0 "U?" H 10500 3154 60  0000 C CNN
-F 1 "7805" H 10350 3550 60  0000 C CNN
-F 2 "" H 10350 3350 60  0000 C CNN
-F 3 "" H 10350 3350 60  0000 C CNN
-	1    10350 3350
-	0    1    1    0
-$EndComp
-Wire Wire Line
-	10400 2500 10400 2950
-Connection ~ 10400 2500
-Wire Wire Line
-	10400 3750 10400 4050
-Wire Wire Line
-	10400 4050 10850 4050
-$Comp
-L GND-RESCUE-leds-controller #PWR?
-U 1 1 570FB4C5
-P 9900 3750
-F 0 "#PWR?" H 9900 3750 30  0001 C CNN
-F 1 "GND" H 9900 3680 30  0001 C CNN
-F 2 "" H 9900 3750 60  0000 C CNN
-F 3 "" H 9900 3750 60  0000 C CNN
-	1    9900 3750
-	1    0    0    -1
-$EndComp
-Wire Wire Line
-	10100 3350 9900 3350
-Wire Wire Line
-	9900 3350 9900 3750
-Text HLabel 10850 4050 2    60   Output ~ 0
-5V
 $EndSCHEMATC
