File: electronics/indus/leds-controller_diy_bare/dcdc_24_12_5.sch (KiCad schematic (older format))
At the start: 20 parts

Commit message: wip bare diy controller - dcdc and refactor
Parts:
- removed C?: 10nF, Capacitors_SMD:C_1206, symbol C-RESCUE-leds-controller
- removed D?: RS1A DIODE, ab2tech:AB2_DO-214AC, symbol DIODE
- removed D?: SMBJ15A Transil, risebox:DIODE_DO_214_AA, symbol ZENER-RESCUE-leds-controller
- gave numbers to parts that had none: 17
Connections:
- wire segments 53 -> 62
