File: electronics/indus/leds-controller_diy_bare/leds-controller.sch (KiCad schematic (older format))
At the start: 19 parts, among them P1 ALIM_12V_60V, P10 THERM_LEDS, P2 MICRO_CTRL, P3 FANS, P4 POT_COLOR2, P5 POT_COLOR3, P6 POT_COLOR4, P7 POT_COLOR1, P8 LED+, P9 LED-

Commit message: footprint with libraries
Parts:
- C21: footprint (none) -> Capacitors_SMD:C_1206
- D1: footprint ab2tech:AB2_DO-214AC -> ab2_passive:AB2_DO-214AC
- R3, R4, R5: footprint (none) -> Resistors_SMD:R_0805
Changed lines of the file:
@@
 F 0 "P1" H 850 1050 50  0000 C CNN
 F 1 "ALIM_12V_60V" V 950 900 50  0000 C CNN
-F 2 "" H 850 900 60  0000 C CNN
+F 2 "" H 850 900 60  0001 C CNN
 F 3 "" H 850 900 60  0000 C CNN
 	1    850  900
@@
 F 0 "P3" H 10800 5700 50  0000 C CNN
 F 1 "FANS" V 10900 5550 50  0000 C CNN
-F 2 "" H 10800 5550 60  0000 C CNN
+F 2 "" H 10800 5550 60  0001 C CNN
 F 3 "" H 10800 5550 60  0000 C CNN
 	1    10800 5550
@@
 F 0 "P7" H 7450 2200 50  0000 C CNN
 F 1 "POT_COLOR1" V 7550 2000 50  0000 C CNN
-F 2 "" H 7450 2000 50  0000 C CNN
+F 2 "" H 7450 2000 50  0001 C CNN
 F 3 "" H 7450 2000 50  0000 C CNN
 	1    7450 2000
@@
 $EndComp
 $Comp
-L GND #PWR9
+L GND #PWR01
 U 1 1 576117B3
 P 7050 2150
-F 0 "#PWR9" H 7050 1900 50  0001 C CNN
+F 0 "#PWR01" H 7050 1900 50  0001 C CNN
 F 1 "GND" H 7050 2000 50  0000 C CNN
 F 2 "" H 7050 2150 50  0000 C CNN
@@
 F 0 "P8" H 10800 2850 50  0000 C CNN
 F 1 "LED+" V 10900 2600 50  0000 C CNN
-F 2 "" H 10800 2600 50  0000 C CNN
+F 2 "" H 10800 2600 50  0001 C CNN
 F 3 "" H 10800 2600 50  0000 C CNN
 	1    10800 2600
@@
 F 0 "P9" H 10800 4150 50  0000 C CNN
 F 1 "LED-" V 10900 3900 50  0000 C CNN
-F 2 "" H 10800 3900 50  0000 C CNN
+F 2 "" H 10800 3900 50  0001 C CNN
 F 3 "" H 10800 3900 50  0000 C CNN
 	1    10800 3900
@@
 F 0 "P4" H 7400 3400 50  0000 C CNN
 F 1 "POT_COLOR2" V 7500 3200 50  0000 C CNN
-F 2 "" H 7400 3200 50  0000 C CNN
+F 2 "" H 7400 3200 50  0001 C CNN
 F 3 "" H 7400 3200 50  0000 C CNN
 	1    7400 3200
@@
 $EndComp
 $Comp
-L GND #PWR6
+L GND #PWR02
 U 1 1 57617728
 P 7000 3350
-F 0 "#PWR6" H 7000 3100 50  0001 C CNN
+F 0 "#PWR02" H 7000 3100 50  0001 C CNN
 F 1 "GND" H 7000 3200 50  0000 C CNN
 F 2 "" H 7000 3350 50  0000 C CNN
@@
 F 0 "P5" H 7400 4600 50  0000 C CNN
 F 1 "POT_COLOR3" V 7500 4400 50  0000 C CNN
-F 2 "" H 7400 4400 50  0000 C CNN
+F 2 "" H 7400 4400 50  0001 C CNN
 F 3 "" H 7400 4400 50  0000 C CNN
 	1    7400 4400
@@
 $EndComp
 $Comp
-L GND #PWR7
+L GND #PWR03
 U 1 1 576178E7
 P 7000 4550
-F 0 "#PWR7" H 7000 4300 50  0001 C CNN
+F 0 "#PWR03" H 7000 4300 50  0001 C CNN
 F 1 "GND" H 7000 4400 50  0000 C CNN
 F 2 "" H 7000 4550 50  0000 C CNN
@@
 F 0 "P6" H 7400 5800 50  0000 C CNN
 F 1 "POT_COLOR4" V 7500 5600 50  0000 C CNN
-F 2 "" H 7400 5600 50  0000 C CNN
+F 2 "" H 7400 5600 50  0001 C CNN
 F 3 "" H 7400 5600 50  0000 C CNN
 	1    7400 5600
@@
 $EndComp
 $Comp
-L GND #PWR8
+L GND #PWR04
 U 1 1 57617AAD
 P 7000 5750
-F 0 "#PWR8" H 7000 5500 50  0001 C CNN
+F 0 "#PWR04" H 7000 5500 50  0001 C CNN
 F 1 "GND" H 7000 5600 50  0000 C CNN
 F 2 "" H 7000 5750 50  0000 C CNN
@@
 F 0 "P2" H 850 5650 50  0000 C CNN
 F 1 "MICRO_CTRL" V 950 5300 50  0000 C CNN
-F 2 "" H 850 5300 50  0000 C CNN
+F 2 "" H 850 5300 50  0001 C CNN
 F 3 "" H 850 5300 50  0000 C CNN
 	1    850  5300
@@
 F 0 "D1" H 1650 1450 40  0000 C CNN
 F 1 "SS16" H 1650 1250 40  0000 C CNN
-F 2 "ab2tech:AB2_DO-214AC" H 1650 1350 60  0001 C CNN
+F 2 "ab2_passive:AB2_DO-214AC" H 1650 1350 60  0001 C CNN
 F 3 "" H 1650 1350 60  0000 C CNN
 	1    1650 1350
@@
 $EndComp
 $Comp
-L GND-RESCUE-leds-controller #PWR3
+L GND-RESCUE-leds-controller #PWR05
 U 1 1 5761ABF9
 P 2050 1900
-F 0 "#PWR3" H 2050 1900 30  0001 C CNN
+F 0 "#PWR05" H 2050 1900 30  0001 C CNN
 F 1 "GND" H 2050 1830 30  0001 C CNN
 F 2 "" H 2050 1900 60  0000 C CNN
@@
 $EndComp
 $Comp
-L GND #PWR2
+L GND #PWR06
 U 1 1 5761F7A3
 P 1450 6000
-F 0 "#PWR2" H 1450 5750 50  0001 C CNN
+F 0 "#PWR06" H 1450 5750 50  0001 C CNN
 F 1 "GND" H 1450 5850 50  0000 C CNN
 F 2 "" H 1450 6000 50  0000 C CNN
@@
 F 0 "P10" H 850 3950 50  0000 C CNN
 F 1 "THERM_LEDS" V 950 3750 50  0000 C CNN
-F 2 "" H 850 3750 50  0000 C CNN
+F 2 "" H 850 3750 50  0001 C CNN
 F 3 "" H 850 3750 50  0000 C CNN
 	1    850  3750
@@
 $EndComp
 $Comp
-L GND #PWR1
+L GND #PWR07
 U 1 1 57631C39
 P 1300 4150
-F 0 "#PWR1" H 1300 3900 50  0001 C CNN
+F 0 "#PWR07" H 1300 3900 50  0001 C CNN
 F 1 "GND" H 1300 4000 50  0000 C CNN
 F 2 "" H 1300 4150 50  0000 C CNN
@@
 PWM_COL4
 $Comp
-L +12V #PWR5
+L +12V #PWR08
 U 1 1 576500F1
 P 5850 1100
-F 0 "#PWR5" H 5850 950 50  0001 C CNN
+F 0 "#PWR08" H 5850 950 50  0001 C CNN
 F 1 "+12V" H 5850 1240 50  0000 C CNN
 F 2 "" H 5850 1100 50  0000 C CNN
@@
 $EndComp
 $Comp
-L +5V #PWR4
+L +5V #PWR09
 U 1 1 57655059
 P 5850 800
-F 0 "#PWR4" H 5850 650 50  0001 C CNN
+F 0 "#PWR09" H 5850 650 50  0001 C CNN
 F 1 "+5V" H 5850 940 50  0000 C CNN
 F 2 "" H 5850 800 50  0000 C CNN
@@
 $EndComp
 $Comp
-L +12V #PWR10
+L +12V #PWR010
 U 1 1 57656258
 P 8750 5650
-F 0 "#PWR10" H 8750 5500 50  0001 C CNN
+F 0 "#PWR010" H 8750 5500 50  0001 C CNN
 F 1 "+12V" H 8750 5790 50  0000 C CNN
 F 2 "" H 8750 5650 50  0000 C CNN
@@
 F 0 "R3" V 1430 5450 50  0000 C CNN
 F 1 "1k" V 1350 5450 50  0000 C CNN
-F 2 "" V 1280 5450 50  0000 C CNN
+F 2 "Resistors_SMD:R_0805" V 1280 5450 50  0001 C CNN
 F 3 "" H 1350 5450 50  0000 C CNN
 	1    1350 5450
@@
 F 0 "R4" V 1430 5550 50  0000 C CNN
 F 1 "1k" V 1350 5550 50  0000 C CNN
-F 2 "" V 1280 5550 50  0000 C CNN
+F 2 "Resistors_SMD:R_0805" V 1280 5550 50  0001 C CNN
 F 3 "" H 1350 5550 50  0000 C CNN
 	1    1350 5550
@@
 F 0 "R5" V 1430 5650 50  0000 C CNN
 F 1 "1k" V 1350 5650 50  0000 C CNN
-F 2 "" V 1280 5650 50  0000 C CNN
+F 2 "Resistors_SMD:R_0805" V 1280 5650 50  0001 C CNN
 F 3 "" H 1350 5650 50  0000 C CNN
 	1    1350 5650
@@
 F 0 "C21" H 2075 4550 50  0000 L CNN
 F 1 "10nF" H 2075 4350 50  0000 L CNN
-F 2 "" H 2088 4300 50  0000 C CNN
+F 2 "Capacitors_SMD:C_1206" H 2088 4300 50  0001 C CNN
 F 3 "" H 2050 4450 50  0000 C CNN
 	1    2050 4450
@@
 $EndComp
 $Comp
-L GND #PWR?
+L GND #PWR011
 U 1 1 576840C0
 P 2450 4700
-F 0 "#PWR?" H 2450 4450 50  0001 C CNN
+F 0 "#PWR011" H 2450 4450 50  0001 C CNN
 F 1 "GND" H 2450 4550 50  0000 C CNN
 F 2 "" H 2450 4700 50  0000 C CNN
