File: electronics/indus/leds-controller_diy_bare/signal_tensions.sch (KiCad schematic (older format))
At the start: 8 parts

Commit message: wip bare diy controller - dcdc and refactor
Parts:
- gave numbers to parts that had none: 8
Changed lines of the file:
@@
 $Descr A4 11693 8268
 encoding utf-8
-Sheet 8 8
+Sheet 8 9
 Title ""
 Date ""
@@
 5V_IN
 $Comp
-L R R?
+L R R34
 U 1 1 57608970
 P 1900 2850
-F 0 "R?" V 1980 2850 50  0000 C CNN
+F 0 "R34" V 1980 2850 50  0000 C CNN
 F 1 "10.2k" V 1900 2850 50  0000 C CNN
 F 2 "" V 1830 2850 50  0000 C CNN
@@
 $EndComp
 $Comp
-L R R?
+L R R35
 U 1 1 576089B7
 P 1900 3550
-F 0 "R?" V 1980 3550 50  0000 C CNN
+F 0 "R35" V 1980 3550 50  0000 C CNN
 F 1 "4.12k" V 1900 3550 50  0000 C CNN
 F 2 "" V 1830 3550 50  0000 C CNN
@@
 $EndComp
 $Comp
-L GND #PWR?
+L GND #PWR025
 U 1 1 576089EA
 P 3100 4800
-F 0 "#PWR?" H 3100 4550 50  0001 C CNN
+F 0 "#PWR025" H 3100 4550 50  0001 C CNN
 F 1 "GND" H 3100 4650 50  0000 C CNN
 F 2 "" H 3100 4800 50  0000 C CNN
@@
 	3100 4200 3100 4800
 $Comp
-L R R?
+L R R36
 U 1 1 57608B16
 P 2700 2850
-F 0 "R?" V 2780 2850 50  0000 C CNN
+F 0 "R36" V 2780 2850 50  0000 C CNN
 F 1 "47.5k" V 2700 2850 50  0000 C CNN
 F 2 "" V 2630 2850 50  0000 C CNN
@@
 $EndComp
 $Comp
-L R R?
+L R R37
 U 1 1 57608B1C
 P 2700 3550
-F 0 "R?" V 2780 3550 50  0000 C CNN
+F 0 "R37" V 2780 3550 50  0000 C CNN
 F 1 "15k" V 2700 3550 50  0000 C CNN
 F 2 "" V 2630 3550 50  0000 C CNN
@@
 	2700 3700 2700 4200
 $Comp
-L R R?
+L R R38
 U 1 1 57608B73
 P 3500 2850
-F 0 "R?" V 3580 2850 50  0000 C CNN
+F 0 "R38" V 3580 2850 50  0000 C CNN
 F 1 "11.5k" V 3500 2850 50  0000 C CNN
 F 2 "" V 3430 2850 50  0000 C CNN
@@
 $EndComp
 $Comp
-L R R?
+L R R39
 U 1 1 57608B79
 P 3500 3550
-F 0 "R?" V 3580 3550 50  0000 C CNN
+F 0 "R39" V 3580 3550 50  0000 C CNN
 F 1 "2.32k" V 3500 3550 50  0000 C CNN
 F 2 "" V 3430 3550 50  0000 C CNN
@@
 Connection ~ 2700 4200
 $Comp
-L R R?
+L R R40
 U 1 1 57608C39
 P 4300 2850
-F 0 "R?" V 4380 2850 50  0000 C CNN
+F 0 "R40" V 4380 2850 50  0000 C CNN
 F 1 "150k" V 4300 2850 50  0000 C CNN
 F 2 "" V 4230 2850 50  0000 C CNN
@@
 $EndComp
 $Comp
-L R R?
+L R R41
 U 1 1 57608C3F
 P 4300 3550
-F 0 "R?" V 4380 3550 50  0000 C CNN
+F 0 "R41" V 4380 3550 50  0000 C CNN
 F 1 "13.7k" V 4300 3550 50  0000 C CNN
 F 2 "" V 4230 3550 50  0000 C CNN

Commit message: footprint with libraries
Parts:
- R34, R35, R36, R37, R38, R39, R40, R41: footprint (none) -> Resistors_SMD:R_0805
Changed lines of the file:
@@
 F 0 "R34" V 1980 2850 50  0000 C CNN
 F 1 "10.2k" V 1900 2850 50  0000 C CNN
-F 2 "" V 1830 2850 50  0000 C CNN
+F 2 "Resistors_SMD:R_0805" V 1830 2850 50  0001 C CNN
 F 3 "" H 1900 2850 50  0000 C CNN
 	1    1900 2850
@@
 F 0 "R35" V 1980 3550 50  0000 C CNN
 F 1 "4.12k" V 1900 3550 50  0000 C CNN
-F 2 "" V 1830 3550 50  0000 C CNN
+F 2 "Resistors_SMD:R_0805" V 1830 3550 50  0001 C CNN
 F 3 "" H 1900 3550 50  0000 C CNN
 	1    1900 3550
@@
 $EndComp
 $Comp
-L GND #PWR16
+L GND #PWR017
 U 1 1 576089EA
 P 3100 4800
-F 0 "#PWR16" H 3100 4550 50  0001 C CNN
+F 0 "#PWR017" H 3100 4550 50  0001 C CNN
 F 1 "GND" H 3100 4650 50  0000 C CNN
 F 2 "" H 3100 4800 50  0000 C CNN
@@
 F 0 "R36" V 2780 2850 50  0000 C CNN
 F 1 "47.5k" V 2700 2850 50  0000 C CNN
-F 2 "" V 2630 2850 50  0000 C CNN
+F 2 "Resistors_SMD:R_0805" V 2630 2850 50  0001 C CNN
 F 3 "" H 2700 2850 50  0000 C CNN
 	1    2700 2850
@@
 F 0 "R37" V 2780 3550 50  0000 C CNN
 F 1 "15k" V 2700 3550 50  0000 C CNN
-F 2 "" V 2630 3550 50  0000 C CNN
+F 2 "Resistors_SMD:R_0805" V 2630 3550 50  0001 C CNN
 F 3 "" H 2700 3550 50  0000 C CNN
 	1    2700 3550
@@
 F 0 "R38" V 3580 2850 50  0000 C CNN
 F 1 "11.5k" V 3500 2850 50  0000 C CNN
-F 2 "" V 3430 2850 50  0000 C CNN
+F 2 "Resistors_SMD:R_0805" V 3430 2850 50  0001 C CNN
 F 3 "" H 3500 2850 50  0000 C CNN
 	1    3500 2850
@@
 F 0 "R39" V 3580 3550 50  0000 C CNN
 F 1 "2.32k" V 3500 3550 50  0000 C CNN
-F 2 "" V 3430 3550 50  0000 C CNN
+F 2 "Resistors_SMD:R_0805" V 3430 3550 50  0001 C CNN
 F 3 "" H 3500 3550 50  0000 C CNN
 	1    3500 3550
@@
 F 0 "R40" V 4380 2850 50  0000 C CNN
 F 1 "150k" V 4300 2850 50  0000 C CNN
-F 2 "" V 4230 2850 50  0000 C CNN
+F 2 "Resistors_SMD:R_0805" V 4230 2850 50  0001 C CNN
 F 3 "" H 4300 2850 50  0000 C CNN
 	1    4300 2850
@@
 F 0 "R41" V 4380 3550 50  0000 C CNN
 F 1 "13.7k" V 4300 3550 50  0000 C CNN
-F 2 "" V 4230 3550 50  0000 C CNN
+F 2 "Resistors_SMD:R_0805" V 4230 3550 50  0001 C CNN
 F 3 "" H 4300 3550 50  0000 C CNN
 	1    4300 3550
