File: electronics/indus/leds-controller_diy_bare/Color1.sch (KiCad schematic (older format))
At the start: 18 parts, among them U4 TPS92513HVDGQT

Commit message: fix some errors
Connections:
- net VIN: now also U4.2 (VIN)
Changed lines of the file:
@@
 POT_OUT
 Wire Wire Line
-	1100 3450 5300 3450
+	1100 3450 5250 3450
 Wire Wire Line
 	1650 4900 10150 4900
@@
 	3550 4750 3550 4900
 Wire Wire Line
-	3550 3550 3550 3450
-Connection ~ 3550 3450
+	3550 3550 3500 3450
+Connection ~ 3500 3450
 Connection ~ 3550 4900
 Wire Wire Line

Commit message: add pinhead footprint
Parts:
- JP1, JP2, JP3, JP4, JP5: footprint (none) -> Connect:PINHEAD1-2
Changed lines of the file:
@@
 F 0 "JP1" H 2400 1150 50  0000 C CNN
 F 1 "M20-9990246" H 2400 920 50  0000 C CNN
-F 2 "" H 2400 1000 50  0001 C CNN
+F 2 "Connect:PINHEAD1-2" H 2400 1000 50  0001 C CNN
 F 3 "" H 2400 1000 50  0000 C CNN
 	1    2400 1000
@@
 F 0 "JP2" H 2400 1500 50  0000 C CNN
 F 1 "M20-9990246" H 2400 1270 50  0000 C CNN
-F 2 "" H 2400 1350 50  0001 C CNN
+F 2 "Connect:PINHEAD1-2" H 2400 1350 50  0001 C CNN
 F 3 "" H 2400 1350 50  0000 C CNN
 	1    2400 1350
@@
 F 0 "JP3" H 2400 1850 50  0000 C CNN
 F 1 "M20-9990246" H 2400 1620 50  0000 C CNN
-F 2 "" H 2400 1700 50  0001 C CNN
+F 2 "Connect:PINHEAD1-2" H 2400 1700 50  0001 C CNN
 F 3 "" H 2400 1700 50  0000 C CNN
 	1    2400 1700
@@
 F 0 "JP4" H 2400 2200 50  0000 C CNN
 F 1 "M20-9990246" H 2400 1970 50  0000 C CNN
-F 2 "" H 2400 2050 50  0001 C CNN
+F 2 "Connect:PINHEAD1-2" H 2400 2050 50  0001 C CNN
 F 3 "" H 2400 2050 50  0000 C CNN
 	1    2400 2050
@@
 F 0 "JP5" H 5650 1600 50  0000 C CNN
 F 1 "M20-9990246" H 5650 1370 50  0000 C CNN
-F 2 "" H 5650 1450 50  0001 C CNN
+F 2 "Connect:PINHEAD1-2" H 5650 1450 50  0001 C CNN
 F 3 "" H 5650 1450 50  0000 C CNN
 	1    5650 1450

Commit message: before routing - no more errors
Changed lines of the file:
@@
 LIBS:contrib
 LIBS:valves
+LIBS:tps54335a
 LIBS:risebox
-LIBS:tps54335a
 LIBS:leds-controller-cache
 EELAYER 25 0
@@
 $EndComp
 $Comp
-L GND-RESCUE-leds-controller #PWR013
+L GND-RESCUE-leds-controller #PWR012
 U 1 1 571557B2
 P 5950 5250
-F 0 "#PWR013" H 5950 5250 30  0001 C CNN
+F 0 "#PWR012" H 5950 5250 30  0001 C CNN
 F 1 "GND" H 5950 5180 30  0001 C CNN
 F 2 "" H 5950 5250 60  0000 C CNN
@@
 	3550 4750 3550 4900
 Wire Wire Line
-	3550 3550 3500 3450
-Connection ~ 3500 3450
+	3550 3550 3550 3450
+Connection ~ 3550 3450
 Connection ~ 3550 4900
 Wire Wire Line

Commit message: added pin with lock footprint
Parts:
- JP1, JP2, JP3, JP4, JP5: footprint Connect:PINHEAD1-2 -> risebox:PINHEAD1-2
Changed lines of the file:
@@
 F 0 "JP1" H 2400 1150 50  0000 C CNN
 F 1 "M20-9990246" H 2400 920 50  0000 C CNN
-F 2 "Connect:PINHEAD1-2" H 2400 1000 50  0001 C CNN
+F 2 "risebox:PINHEAD1-2" H 2400 1000 50  0001 C CNN
 F 3 "" H 2400 1000 50  0000 C CNN
 	1    2400 1000
@@
 F 0 "JP2" H 2400 1500 50  0000 C CNN
 F 1 "M20-9990246" H 2400 1270 50  0000 C CNN
-F 2 "Connect:PINHEAD1-2" H 2400 1350 50  0001 C CNN
+F 2 "risebox:PINHEAD1-2" H 2400 1350 50  0001 C CNN
 F 3 "" H 2400 1350 50  0000 C CNN
 	1    2400 1350
@@
 F 0 "JP3" H 2400 1850 50  0000 C CNN
 F 1 "M20-9990246" H 2400 1620 50  0000 C CNN
-F 2 "Connect:PINHEAD1-2" H 2400 1700 50  0001 C CNN
+F 2 "risebox:PINHEAD1-2" H 2400 1700 50  0001 C CNN
 F 3 "" H 2400 1700 50  0000 C CNN
 	1    2400 1700
@@
 F 0 "JP4" H 2400 2200 50  0000 C CNN
 F 1 "M20-9990246" H 2400 1970 50  0000 C CNN
-F 2 "Connect:PINHEAD1-2" H 2400 2050 50  0001 C CNN
+F 2 "risebox:PINHEAD1-2" H 2400 2050 50  0001 C CNN
 F 3 "" H 2400 2050 50  0000 C CNN
 	1    2400 2050
@@
 F 0 "JP5" H 5650 1600 50  0000 C CNN
 F 1 "M20-9990246" H 5650 1370 50  0000 C CNN
-F 2 "Connect:PINHEAD1-2" H 5650 1450 50  0001 C CNN
+F 2 "risebox:PINHEAD1-2" H 5650 1450 50  0001 C CNN
 F 3 "" H 5650 1450 50  0000 C CNN
 	1    5650 1450
