File: electronics/indus/leds-controller_diy_bare/Color2.sch (KiCad schematic (older format))
At the start: 18 parts, among them U1 TPS92513HVDGQT

Commit message: added pin with lock footprint
Parts:
- JP10, JP6, JP7, JP8, JP9: footprint Connect:PINHEAD1-2 -> risebox:PINHEAD1-2
Changed lines of the file:
@@
 F 0 "JP6" H 2500 1650 50  0000 C CNN
 F 1 "M20-9990246" H 2500 1420 50  0000 C CNN
-F 2 "Connect:PINHEAD1-2" H 2500 1500 50  0001 C CNN
+F 2 "risebox:PINHEAD1-2" H 2500 1500 50  0001 C CNN
 F 3 "" H 2500 1500 50  0000 C CNN
 	1    2500 1500
@@
 F 0 "JP7" H 2500 2000 50  0000 C CNN
 F 1 "M20-9990246" H 2500 1770 50  0000 C CNN
-F 2 "Connect:PINHEAD1-2" H 2500 1850 50  0001 C CNN
+F 2 "risebox:PINHEAD1-2" H 2500 1850 50  0001 C CNN
 F 3 "" H 2500 1850 50  0000 C CNN
 	1    2500 1850
@@
 F 0 "JP8" H 2500 2350 50  0000 C CNN
 F 1 "M20-9990246" H 2500 2120 50  0000 C CNN
-F 2 "Connect:PINHEAD1-2" H 2500 2200 50  0001 C CNN
+F 2 "risebox:PINHEAD1-2" H 2500 2200 50  0001 C CNN
 F 3 "" H 2500 2200 50  0000 C CNN
 	1    2500 2200
@@
 F 0 "JP9" H 2500 2700 50  0000 C CNN
 F 1 "M20-9990246" H 2500 2470 50  0000 C CNN
-F 2 "Connect:PINHEAD1-2" H 2500 2550 50  0001 C CNN
+F 2 "risebox:PINHEAD1-2" H 2500 2550 50  0001 C CNN
 F 3 "" H 2500 2550 50  0000 C CNN
 	1    2500 2550
@@
 F 0 "JP10" H 5750 2100 50  0000 C CNN
 F 1 "M20-9990246" H 5750 1870 50  0000 C CNN
-F 2 "Connect:PINHEAD1-2" H 5750 1950 50  0001 C CNN
+F 2 "risebox:PINHEAD1-2" H 5750 1950 50  0001 C CNN
 F 3 "" H 5750 1950 50  0000 C CNN
 	1    5750 1950
