File: electronics/indus/leds-controller_diy_bare/Color3.sch (KiCad schematic (older format))
At the start: 18 parts, among them U2 TPS92513HVDGQT

Commit message: added pin with lock footprint
Parts:
- JP11, JP12, JP13, JP14, JP15: footprint Connect:PINHEAD1-2 -> risebox:PINHEAD1-2
Changed lines of the file:
@@
 F 0 "JP11" H 2500 1550 50  0000 C CNN
 F 1 "M20-9990246" H 2500 1320 50  0000 C CNN
-F 2 "Connect:PINHEAD1-2" H 2500 1400 50  0001 C CNN
+F 2 "risebox:PINHEAD1-2" H 2500 1400 50  0001 C CNN
 F 3 "" H 2500 1400 50  0000 C CNN
 	1    2500 1400
@@
 F 0 "JP12" H 2500 1900 50  0000 C CNN
 F 1 "M20-9990246" H 2500 1670 50  0000 C CNN
-F 2 "Connect:PINHEAD1-2" H 2500 1750 50  0001 C CNN
+F 2 "risebox:PINHEAD1-2" H 2500 1750 50  0001 C CNN
 F 3 "" H 2500 1750 50  0000 C CNN
 	1    2500 1750
@@
 F 0 "JP13" H 2500 2250 50  0000 C CNN
 F 1 "M20-9990246" H 2500 2020 50  0000 C CNN
-F 2 "Connect:PINHEAD1-2" H 2500 2100 50  0001 C CNN
+F 2 "risebox:PINHEAD1-2" H 2500 2100 50  0001 C CNN
 F 3 "" H 2500 2100 50  0000 C CNN
 	1    2500 2100
@@
 F 0 "JP14" H 2500 2600 50  0000 C CNN
 F 1 "M20-9990246" H 2500 2370 50  0000 C CNN
-F 2 "Connect:PINHEAD1-2" H 2500 2450 50  0001 C CNN
+F 2 "risebox:PINHEAD1-2" H 2500 2450 50  0001 C CNN
 F 3 "" H 2500 2450 50  0000 C CNN
 	1    2500 2450
@@
 F 0 "JP15" H 5750 2000 50  0000 C CNN
 F 1 "M20-9990246" H 5750 1770 50  0000 C CNN
-F 2 "Connect:PINHEAD1-2" H 5750 1850 50  0001 C CNN
+F 2 "risebox:PINHEAD1-2" H 5750 1850 50  0001 C CNN
 F 3 "" H 5750 1850 50  0000 C CNN
 	1    5750 1850
