File: electronics/indus/leds-controller_diy_bare/Color4.sch (KiCad schematic (older format))
At the start: 18 parts, among them U3 TPS92513HVDGQT

Commit message: added pin with lock footprint
Parts:
- JP16, JP17, JP18, JP19, JP20: footprint Connect:PINHEAD1-2 -> risebox:PINHEAD1-2
Changed lines of the file:
@@
 F 0 "JP16" H 2550 1700 50  0000 C CNN
 F 1 "M20-9990246" H 2550 1470 50  0000 C CNN
-F 2 "Connect:PINHEAD1-2" H 2550 1550 50  0001 C CNN
+F 2 "risebox:PINHEAD1-2" H 2550 1550 50  0001 C CNN
 F 3 "" H 2550 1550 50  0000 C CNN
 	1    2550 1550
@@
 F 0 "JP17" H 2550 2050 50  0000 C CNN
 F 1 "M20-9990246" H 2550 1820 50  0000 C CNN
-F 2 "Connect:PINHEAD1-2" H 2550 1900 50  0001 C CNN
+F 2 "risebox:PINHEAD1-2" H 2550 1900 50  0001 C CNN
 F 3 "" H 2550 1900 50  0000 C CNN
 	1    2550 1900
@@
 F 0 "JP18" H 2550 2400 50  0000 C CNN
 F 1 "M20-9990246" H 2550 2170 50  0000 C CNN
-F 2 "Connect:PINHEAD1-2" H 2550 2250 50  0001 C CNN
+F 2 "risebox:PINHEAD1-2" H 2550 2250 50  0001 C CNN
 F 3 "" H 2550 2250 50  0000 C CNN
 	1    2550 2250
@@
 F 0 "JP19" H 2550 2750 50  0000 C CNN
 F 1 "M20-9990246" H 2550 2520 50  0000 C CNN
-F 2 "Connect:PINHEAD1-2" H 2550 2600 50  0001 C CNN
+F 2 "risebox:PINHEAD1-2" H 2550 2600 50  0001 C CNN
 F 3 "" H 2550 2600 50  0000 C CNN
 	1    2550 2600
@@
 F 0 "JP20" H 5800 2150 50  0000 C CNN
 F 1 "M20-9990246" H 5800 1920 50  0000 C CNN
-F 2 "Connect:PINHEAD1-2" H 5800 2000 50  0001 C CNN
+F 2 "risebox:PINHEAD1-2" H 5800 2000 50  0001 C CNN
 F 3 "" H 5800 2000 50  0000 C CNN
 	1    5800 2000
