File: electronics/indus/leds_diy/leds.sch (KiCad schematic (older format))
At the start: 21 parts, among them P1 LED+, P2 THERM, P3 LED-

Commit message: wip bare diy controller
Parts:
- D1, D10, D11, D12, D13, D14, D15, D16, D2, D3, D4, D5, D6, D7, D8, D9: symbol LED -> LED-RESCUE-leds
- R1: symbol R -> R-RESCUE-leds
Changed lines of the file:
@@
 EESchema Schematic File Version 2
+LIBS:leds-rescue
 LIBS:power
 LIBS:device
@@
 LIBS:memory
 LIBS:xilinx
-LIBS:special
 LIBS:microcontrollers
 LIBS:dsp
@@
 $EndDescr
 $Comp
-L LED D1
+L LED-RESCUE-leds D1
 U 1 1 56E1A1EF
 P 4750 1950
@@
 $EndComp
 $Comp
-L LED D5
+L LED-RESCUE-leds D5
 U 1 1 56E1A231
 P 5400 1950
@@
 $EndComp
 $Comp
-L LED D9
+L LED-RESCUE-leds D9
 U 1 1 56E1A294
 P 6050 1950
@@
 $EndComp
 $Comp
-L LED D13
+L LED-RESCUE-leds D13
 U 1 1 56E1A2C5
 P 6700 1950
@@
 $EndComp
 $Comp
-L LED D2
+L LED-RESCUE-leds D2
 U 1 1 56E1BEDB
 P 4750 2450
@@
 $EndComp
 $Comp
-L LED D6
+L LED-RESCUE-leds D6
 U 1 1 56E1BEE1
 P 5400 2450
@@
 $EndComp
 $Comp
-L LED D10
+L LED-RESCUE-leds D10
 U 1 1 56E1BEE7
 P 6050 2450
@@
 $EndComp
 $Comp
-L LED D14
+L LED-RESCUE-leds D14
 U 1 1 56E1BEED
 P 6700 2450
@@
 $EndComp
 $Comp
-L LED D3
+L LED-RESCUE-leds D3
 U 1 1 56E1C418
 P 4750 2950
@@
 $EndComp
 $Comp
-L LED D7
+L LED-RESCUE-leds D7
 U 1 1 56E1C41E
 P 5400 2950
@@
 $EndComp
 $Comp
-L LED D11
+L LED-RESCUE-leds D11
 U 1 1 56E1C424
 P 6050 2950
@@
 $EndComp
 $Comp
-L LED D15
+L LED-RESCUE-leds D15
 U 1 1 56E1C42A
 P 6700 2950
@@
 $EndComp
 $Comp
-L LED D4
+L LED-RESCUE-leds D4
 U 1 1 56E1C44F
 P 4750 3450
@@
 $EndComp
 $Comp
-L LED D8
+L LED-RESCUE-leds D8
 U 1 1 56E1C455
 P 5400 3450
@@
 $EndComp
 $Comp
-L LED D12
+L LED-RESCUE-leds D12
 U 1 1 56E1C45B
 P 6050 3450
@@
 $EndComp
 $Comp
-L LED D16
+L LED-RESCUE-leds D16
 U 1 1 56E1C461
 P 6700 3450
@@
 	5000 4550 5000 4800
 $Comp
-L GND #PWR01
+L GND-RESCUE-leds #PWR1
 U 1 1 5714EE15
 P 6050 5200
-F 0 "#PWR01" H 6050 5200 30  0001 C CNN
+F 0 "#PWR1" H 6050 5200 30  0001 C CNN
 F 1 "GND" H 6050 5130 30  0001 C CNN
 F 2 "" H 6050 5200 60  0000 C CNN
@@
 	5100 4700 7100 4700
 $Comp
-L R R1
+L R-RESCUE-leds R1
 U 1 1 574515E8
 P 5550 4400

Commit message: updated LEDS footprint & TH ref
Parts:
- D1, D10, D11, D12, D13, D14, D15, D16, D2, D3, D4, D5, D6, D7, D8, D9: footprint (none) -> w_smd_leds:Luxeon_C
- P2: footprint (none) -> risebox:THERM_NTCS0603E3272JMT_SMD0603
- R1: value 10K -> 2.7K
- TH1: value THERM CTN 10K -> MC01W080512K7
Changed lines of the file:
@@
 F 0 "D1" H 4750 2050 50  0000 C CNN
 F 1 "LED" H 4750 1850 50  0000 C CNN
-F 2 "" H 4750 1950 60  0000 C CNN
+F 2 "w_smd_leds:Luxeon_C" H 4750 1950 60  0001 C CNN
 F 3 "" H 4750 1950 60  0000 C CNN
 	1    4750 1950
@@
 F 0 "D5" H 5400 2050 50  0000 C CNN
 F 1 "LED" H 5400 1850 50  0000 C CNN
-F 2 "" H 5400 1950 60  0000 C CNN
+F 2 "w_smd_leds:Luxeon_C" H 5400 1950 60  0001 C CNN
 F 3 "" H 5400 1950 60  0000 C CNN
 	1    5400 1950
@@
 F 0 "D9" H 6050 2050 50  0000 C CNN
 F 1 "LED" H 6050 1850 50  0000 C CNN
-F 2 "" H 6050 1950 60  0000 C CNN
+F 2 "w_smd_leds:Luxeon_C" H 6050 1950 60  0001 C CNN
 F 3 "" H 6050 1950 60  0000 C CNN
 	1    6050 1950
@@
 F 0 "D13" H 6700 2050 50  0000 C CNN
 F 1 "LED" H 6700 1850 50  0000 C CNN
-F 2 "" H 6700 1950 60  0000 C CNN
+F 2 "w_smd_leds:Luxeon_C" H 6700 1950 60  0001 C CNN
 F 3 "" H 6700 1950 60  0000 C CNN
 	1    6700 1950
@@
 F 0 "D2" H 4750 2550 50  0000 C CNN
 F 1 "LED" H 4750 2350 50  0000 C CNN
-F 2 "" H 4750 2450 60  0000 C CNN
+F 2 "w_smd_leds:Luxeon_C" H 4750 2450 60  0001 C CNN
 F 3 "" H 4750 2450 60  0000 C CNN
 	1    4750 2450
@@
 F 0 "D6" H 5400 2550 50  0000 C CNN
 F 1 "LED" H 5400 2350 50  0000 C CNN
-F 2 "" H 5400 2450 60  0000 C CNN
+F 2 "w_smd_leds:Luxeon_C" H 5400 2450 60  0001 C CNN
 F 3 "" H 5400 2450 60  0000 C CNN
 	1    5400 2450
@@
 F 0 "D10" H 6050 2550 50  0000 C CNN
 F 1 "LED" H 6050 2350 50  0000 C CNN
-F 2 "" H 6050 2450 60  0000 C CNN
+F 2 "w_smd_leds:Luxeon_C" H 6050 2450 60  0001 C CNN
 F 3 "" H 6050 2450 60  0000 C CNN
 	1    6050 2450
@@
 F 0 "D14" H 6700 2550 50  0000 C CNN
 F 1 "LED" H 6700 2350 50  0000 C CNN
-F 2 "" H 6700 2450 60  0000 C CNN
+F 2 "w_smd_leds:Luxeon_C" H 6700 2450 60  0001 C CNN
 F 3 "" H 6700 2450 60  0000 C CNN
 	1    6700 2450
@@
 F 0 "D3" H 4750 3050 50  0000 C CNN
 F 1 "LED" H 4750 2850 50  0000 C CNN
-F 2 "" H 4750 2950 60  0000 C CNN
+F 2 "w_smd_leds:Luxeon_C" H 4750 2950 60  0001 C CNN
 F 3 "" H 4750 2950 60  0000 C CNN
 	1    4750 2950
@@
 F 0 "D7" H 5400 3050 50  0000 C CNN
 F 1 "LED" H 5400 2850 50  0000 C CNN
-F 2 "" H 5400 2950 60  0000 C CNN
+F 2 "w_smd_leds:Luxeon_C" H 5400 2950 60  0001 C CNN
 F 3 "" H 5400 2950 60  0000 C CNN
 	1    5400 2950
@@
 F 0 "D11" H 6050 3050 50  0000 C CNN
 F 1 "LED" H 6050 2850 50  0000 C CNN
-F 2 "" H 6050 2950 60  0000 C CNN
+F 2 "w_smd_leds:Luxeon_C" H 6050 2950 60  0001 C CNN
 F 3 "" H 6050 2950 60  0000 C CNN
 	1    6050 2950
@@
 F 0 "D15" H 6700 3050 50  0000 C CNN
 F 1 "LED" H 6700 2850 50  0000 C CNN
-F 2 "" H 6700 2950 60  0000 C CNN
+F 2 "w_smd_leds:Luxeon_C" H 6700 2950 60  0001 C CNN
 F 3 "" H 6700 2950 60  0000 C CNN
 	1    6700 2950
@@
 F 0 "D4" H 4750 3550 50  0000 C CNN
 F 1 "LED" H 4750 3350 50  0000 C CNN
-F 2 "" H 4750 3450 60  0000 C CNN
+F 2 "w_smd_leds:Luxeon_C" H 4750 3450 60  0001 C CNN
 F 3 "" H 4750 3450 60  0000 C CNN
 	1    4750 3450
@@
 F 0 "D8" H 5400 3550 50  0000 C CNN
 F 1 "LED" H 5400 3350 50  0000 C CNN
-F 2 "" H 5400 3450 60  0000 C CNN
+F 2 "w_smd_leds:Luxeon_C" H 5400 3450 60  0001 C CNN
 F 3 "" H 5400 3450 60  0000 C CNN
 	1    5400 3450
@@
 F 0 "D12" H 6050 3550 50  0000 C CNN
 F 1 "LED" H 6050 3350 50  0000 C CNN
-F 2 "" H 6050 3450 60  0000 C CNN
+F 2 "w_smd_leds:Luxeon_C" H 6050 3450 60  0001 C CNN
 F 3 "" H 6050 3450 60  0000 C CNN
 	1    6050 3450
@@
 F 0 "D16" H 6700 3550 50  0000 C CNN
 F 1 "LED" H 6700 3350 50  0000 C CNN
-F 2 "" H 6700 3450 60  0000 C CNN
+F 2 "w_smd_leds:Luxeon_C" H 6700 3450 60  0001 C CNN
 F 3 "" H 6700 3450 60  0000 C CNN
 	1    6700 3450
@@
 P 6550 4400
 F 0 "TH1" V 6650 4450 50  0000 C CNN
-F 1 "THERM CTN 10K" V 6450 4400 50  0000 C CNN
-F 2 "" H 6550 4400 60  0000 C CNN
+F 1 "MC01W080512K7" V 6450 4400 50  0000 C CNN
+F 2 "" H 6550 4400 60  0001 C CNN
 F 3 "" H 6550 4400 60  0000 C CNN
 	1    6550 4400
@@
 	5000 4550 5000 4800
 $Comp
-L GND-RESCUE-leds #PWR1
+L GND-RESCUE-leds #PWR01
 U 1 1 5714EE15
 P 6050 5200
-F 0 "#PWR1" H 6050 5200 30  0001 C CNN
+F 0 "#PWR01" H 6050 5200 30  0001 C CNN
 F 1 "GND" H 6050 5130 30  0001 C CNN
 F 2 "" H 6050 5200 60  0000 C CNN
@@
 P 5550 4400
 F 0 "R1" V 5630 4400 40  0000 C CNN
-F 1 "10K" V 5557 4401 40  0000 C CNN
-F 2 "" V 5480 4400 30  0000 C CNN
+F 1 "2.7K" V 5557 4401 40  0000 C CNN
+F 2 "" V 5480 4400 30  0001 C CNN
 F 3 "" H 5550 4400 30  0000 C CNN
 	1    5550 4400
@@
 F 0 "P1" H 1950 3000 50  0000 C CNN
 F 1 "LED+" V 2050 2750 50  0000 C CNN
-F 2 "" H 1950 2750 60  0000 C CNN
+F 2 "" H 1950 2750 60  0001 C CNN
 F 3 "" H 1950 2750 60  0000 C CNN
 	1    1950 2750
@@
 F 0 "P3" H 9200 2950 50  0000 C CNN
 F 1 "LED-" V 9300 2700 50  0000 C CNN
-F 2 "" H 9200 2700 60  0000 C CNN
+F 2 "" H 9200 2700 60  0001 C CNN
 F 3 "" H 9200 2700 60  0000 C CNN
 	1    9200 2700
@@
 F 0 "P2" H 5000 5200 50  0000 C CNN
 F 1 "THERM" V 5100 5000 50  0000 C CNN
-F 2 "" H 5000 5000 60  0000 C CNN
+F 2 "risebox:THERM_NTCS0603E3272JMT_SMD0603" H 5000 5000 60  0001 C CNN
 F 3 "" H 5000 5000 60  0000 C CNN
 	1    5000 5000

Commit message: first routing of led
Parts:
- D1, D10, D11, D12, D13, D14, D15, D16, D2, D3, D4, D5, D6, D7, D8, D9: footprint w_smd_leds:Luxeon_C -> risebox:LUXEON-C
- P1, P3: footprint (none) -> risebox:PINHEAD_LOCK_1-4
- P2: footprint risebox:THERM_NTCS0603E3272JMT_SMD0603 -> risebox:PINHEAD_LOCK_1-3
- R1: footprint (none) -> Resistors_SMD:R_0805
- TH1: value MC01W080512K7 -> NTCS0603E3272JMT; footprint (none) -> risebox:THERM_NTCS0603E3272JMT_SMD0603
Changed lines of the file:
@@
 F 0 "D1" H 4750 2050 50  0000 C CNN
 F 1 "LED" H 4750 1850 50  0000 C CNN
-F 2 "w_smd_leds:Luxeon_C" H 4750 1950 60  0001 C CNN
+F 2 "risebox:LUXEON-C" H 4750 1950 60  0001 C CNN
 F 3 "" H 4750 1950 60  0000 C CNN
 	1    4750 1950
@@
 F 0 "D5" H 5400 2050 50  0000 C CNN
 F 1 "LED" H 5400 1850 50  0000 C CNN
-F 2 "w_smd_leds:Luxeon_C" H 5400 1950 60  0001 C CNN
+F 2 "risebox:LUXEON-C" H 5400 1950 60  0001 C CNN
 F 3 "" H 5400 1950 60  0000 C CNN
 	1    5400 1950
@@
 F 0 "D9" H 6050 2050 50  0000 C CNN
 F 1 "LED" H 6050 1850 50  0000 C CNN
-F 2 "w_smd_leds:Luxeon_C" H 6050 1950 60  0001 C CNN
+F 2 "risebox:LUXEON-C" H 6050 1950 60  0001 C CNN
 F 3 "" H 6050 1950 60  0000 C CNN
 	1    6050 1950
@@
 F 0 "D13" H 6700 2050 50  0000 C CNN
 F 1 "LED" H 6700 1850 50  0000 C CNN
-F 2 "w_smd_leds:Luxeon_C" H 6700 1950 60  0001 C CNN
+F 2 "risebox:LUXEON-C" H 6700 1950 60  0001 C CNN
 F 3 "" H 6700 1950 60  0000 C CNN
 	1    6700 1950
@@
 F 0 "D2" H 4750 2550 50  0000 C CNN
 F 1 "LED" H 4750 2350 50  0000 C CNN
-F 2 "w_smd_leds:Luxeon_C" H 4750 2450 60  0001 C CNN
+F 2 "risebox:LUXEON-C" H 4750 2450 60  0001 C CNN
 F 3 "" H 4750 2450 60  0000 C CNN
 	1    4750 2450
@@
 F 0 "D6" H 5400 2550 50  0000 C CNN
 F 1 "LED" H 5400 2350 50  0000 C CNN
-F 2 "w_smd_leds:Luxeon_C" H 5400 2450 60  0001 C CNN
+F 2 "risebox:LUXEON-C" H 5400 2450 60  0001 C CNN
 F 3 "" H 5400 2450 60  0000 C CNN
 	1    5400 2450
@@
 F 0 "D10" H 6050 2550 50  0000 C CNN
 F 1 "LED" H 6050 2350 50  0000 C CNN
-F 2 "w_smd_leds:Luxeon_C" H 6050 2450 60  0001 C CNN
+F 2 "risebox:LUXEON-C" H 6050 2450 60  0001 C CNN
 F 3 "" H 6050 2450 60  0000 C CNN
 	1    6050 2450
@@
 F 0 "D14" H 6700 2550 50  0000 C CNN
 F 1 "LED" H 6700 2350 50  0000 C CNN
-F 2 "w_smd_leds:Luxeon_C" H 6700 2450 60  0001 C CNN
+F 2 "risebox:LUXEON-C" H 6700 2450 60  0001 C CNN
 F 3 "" H 6700 2450 60  0000 C CNN
 	1    6700 2450
@@
 F 0 "D3" H 4750 3050 50  0000 C CNN
 F 1 "LED" H 4750 2850 50  0000 C CNN
-F 2 "w_smd_leds:Luxeon_C" H 4750 2950 60  0001 C CNN
+F 2 "risebox:LUXEON-C" H 4750 2950 60  0001 C CNN
 F 3 "" H 4750 2950 60  0000 C CNN
 	1    4750 2950
@@
 F 0 "D7" H 5400 3050 50  0000 C CNN
 F 1 "LED" H 5400 2850 50  0000 C CNN
-F 2 "w_smd_leds:Luxeon_C" H 5400 2950 60  0001 C CNN
+F 2 "risebox:LUXEON-C" H 5400 2950 60  0001 C CNN
 F 3 "" H 5400 2950 60  0000 C CNN
 	1    5400 2950
@@
 F 0 "D11" H 6050 3050 50  0000 C CNN
 F 1 "LED" H 6050 2850 50  0000 C CNN
-F 2 "w_smd_leds:Luxeon_C" H 6050 2950 60  0001 C CNN
+F 2 "risebox:LUXEON-C" H 6050 2950 60  0001 C CNN
 F 3 "" H 6050 2950 60  0000 C CNN
 	1    6050 2950
@@
 F 0 "D15" H 6700 3050 50  0000 C CNN
 F 1 "LED" H 6700 2850 50  0000 C CNN
-F 2 "w_smd_leds:Luxeon_C" H 6700 2950 60  0001 C CNN
+F 2 "risebox:LUXEON-C" H 6700 2950 60  0001 C CNN
 F 3 "" H 6700 2950 60  0000 C CNN
 	1    6700 2950
@@
 F 0 "D4" H 4750 3550 50  0000 C CNN
 F 1 "LED" H 4750 3350 50  0000 C CNN
-F 2 "w_smd_leds:Luxeon_C" H 4750 3450 60  0001 C CNN
+F 2 "risebox:LUXEON-C" H 4750 3450 60  0001 C CNN
 F 3 "" H 4750 3450 60  0000 C CNN
 	1    4750 3450
@@
 F 0 "D8" H 5400 3550 50  0000 C CNN
 F 1 "LED" H 5400 3350 50  0000 C CNN
-F 2 "w_smd_leds:Luxeon_C" H 5400 3450 60  0001 C CNN
+F 2 "risebox:LUXEON-C" H 5400 3450 60  0001 C CNN
 F 3 "" H 5400 3450 60  0000 C CNN
 	1    5400 3450
@@
 F 0 "D12" H 6050 3550 50  0000 C CNN
 F 1 "LED" H 6050 3350 50  0000 C CNN
-F 2 "w_smd_leds:Luxeon_C" H 6050 3450 60  0001 C CNN
+F 2 "risebox:LUXEON-C" H 6050 3450 60  0001 C CNN
 F 3 "" H 6050 3450 60  0000 C CNN
 	1    6050 3450
@@
 F 0 "D16" H 6700 3550 50  0000 C CNN
 F 1 "LED" H 6700 3350 50  0000 C CNN
-F 2 "w_smd_leds:Luxeon_C" H 6700 3450 60  0001 C CNN
+F 2 "risebox:LUXEON-C" H 6700 3450 60  0001 C CNN
 F 3 "" H 6700 3450 60  0000 C CNN
 	1    6700 3450
@@
 P 6550 4400
 F 0 "TH1" V 6650 4450 50  0000 C CNN
-F 1 "MC01W080512K7" V 6450 4400 50  0000 C CNN
-F 2 "" H 6550 4400 60  0001 C CNN
+F 1 "NTCS0603E3272JMT" V 6450 4400 50  0000 C CNN
+F 2 "risebox:THERM_NTCS0603E3272JMT_SMD0603" H 6550 4400 60  0001 C CNN
 F 3 "" H 6550 4400 60  0000 C CNN
 	1    6550 4400
@@
 F 0 "R1" V 5630 4400 40  0000 C CNN
 F 1 "2.7K" V 5557 4401 40  0000 C CNN
-F 2 "" V 5480 4400 30  0001 C CNN
+F 2 "Resistors_SMD:R_0805" V 5480 4400 30  0001 C CNN
 F 3 "" H 5550 4400 30  0000 C CNN
 	1    5550 4400
@@
 F 0 "P1" H 1950 3000 50  0000 C CNN
 F 1 "LED+" V 2050 2750 50  0000 C CNN
-F 2 "" H 1950 2750 60  0001 C CNN
+F 2 "risebox:PINHEAD_LOCK_1-4" H 1950 2750 60  0001 C CNN
 F 3 "" H 1950 2750 60  0000 C CNN
 	1    1950 2750
@@
 F 0 "P3" H 9200 2950 50  0000 C CNN
 F 1 "LED-" V 9300 2700 50  0000 C CNN
-F 2 "" H 9200 2700 60  0001 C CNN
+F 2 "risebox:PINHEAD_LOCK_1-4" H 9200 2700 60  0001 C CNN
 F 3 "" H 9200 2700 60  0000 C CNN
 	1    9200 2700
@@
 F 0 "P2" H 5000 5200 50  0000 C CNN
 F 1 "THERM" V 5100 5000 50  0000 C CNN
-F 2 "risebox:THERM_NTCS0603E3272JMT_SMD0603" H 5000 5000 60  0001 C CNN
+F 2 "risebox:PINHEAD_LOCK_1-3" H 5000 5000 60  0001 C CNN
 F 3 "" H 5000 5000 60  0000 C CNN
 	1    5000 5000
